File: PCBs/XDS100v2 Programmer/XDS100v2 Programmer.sch (KiCad schematic (older format))
At the start: 0 parts

Commit message: Schematic Complete
- Completed Full Schematic
- Completed BOM
- Some footprints selected
Parts:
- added C1, C2: 4.7uF, Capacitors_SMD:C_0805, symbol Device:C_Small
- added C10, C11, C5, C6, C7, C8: 0.1uF, Capacitors_SMD:C_0805, symbol Device:C_Small
- added C12, C13: 36p, Capacitors_SMD:C_0603, symbol Device:C_Small
- added C3: 1uF, Capacitors_SMD:C_0805, symbol Device:C_Small
- added C4: 100uF, symbol Device:CP
- added C9: 3.3uF, Capacitors_SMD:C_0805, symbol Device:C_Small
- added D1, D2, D3: LED, LEDs:LED_0805, symbol Device:LED
- added F1: 500mA, symbol Device:Fuse
- added H? (x6): MountingHole_Pad, symbol Mechanical:MountingHole_Pad
- added J1: USB_B_Mini, symbol Connector:USB_B_Mini
- added J2: Conn_02x05, symbol Connector_Generic:Conn_02x05_Counter_Clockwise
- added L1, L2: FB, Inductors_SMD:L_0402, symbol Device:L
- added R1, R3, R4: 1k, Resistors_SMD:R_0805, symbol Device:R_Small_US
- added R10, R13, R14, R15, R5: 2.2k, Resistors_SMD:R_0805, symbol Device:R_Small_US
- added R11, R12: 820, Resistors_SMD:R_0805, symbol Device:R_Small_US
- added R2, R7: 10k, Resistors_SMD:R_0805, symbol Device:R_Small_US
- added R6: 12k, Resistors_SMD:R_0805, symbol Device:R_Small_US
- added R8, R9: 330, Resistors_SMD:R_0805, symbol Device:R_Small_US
- added SW1, SW2: SW_DIP_x02, symbol Switch:SW_DIP_x02
- added SW3: SW_DIP_x03, symbol Switch:SW_DIP_x03
- added U1: TLV1117-33, TO_SOT_Packages_SMD:SOT-223, symbol Regulator_Linear:TLV1117-33
- added U2: ISO7240, Housings_SOIC:SOIC-16W_7.5x10.3mm_Pitch1.27mm, symbol XDS100v2~Programmer:ISO7240
- added U3: EEPROM_Array, TO_SOT_Packages_SMD:SOT-23-6, symbol XDS100v2~Programmer:EEPROM_Array
- added U4: FT2232H, Housings_DFN_QFN:QFN-64-1EP_9x9mm_Pitch0.5mm, symbol Interface_USB:FT2232H
- added U5: ISO7231, Housings_SOIC:SOIC-16W_7.5x10.3mm_Pitch1.27mm, symbol XDS100v2~Programmer:ISO7231
- added U6: EEPROM_Array_8pin, symbol XDS100v2~Programmer:EEPROM_Array_8pin
- added Y1: 12MHz, symbol Device:Crystal_Small
Connections:
- net labels added: +1V8, +3V3, +5V, 3V3_MCU, D+, D-, FTDI_CLK, FTDI_CS, FTDI_DATA, GND, GNDD, GPIO28, GPIO29, GPIO34, JTAG_TRST, SCI_RX, SCI_TX, TCK, TDI, TDO, TMS, TRST, ~PWREN~, ~SUSPEND~
- wire segments 0 -> 266
- no-connect marks 0 -> 25
Other:
- note added: "Duplicate incase 8pin EEPROM does not work"

Commit message: Selected Footprints
- Created and assigned all required footprints
Parts:
- C4: footprint (none) -> Capacitors_Tantalum_SMD:CP_Tantalum_Case-U_EIA-6032-15_Reflow
- F1: footprint (none) -> XDS100v2 Programmer:1812_PloyFuse
- H1, H2, H3, H4, H5, H6: renamed from H?; footprint (none) -> Mounting_Holes:MountingHole_3mm_Pad_Via
- J1: footprint (none) -> XDS100v2 Programmer:USB_Mini_B_32005-201
- J2: footprint (none) -> Pin_Headers:Pin_Header_Straight_2x05_Pitch2.54mm
- SW1, SW2: footprint (none) -> XDS100v2 Programmer:CTS_DPST_Switch
- SW3: footprint (none) -> XDS100v2 Programmer:CTS_3DIP_Switch
- U6: footprint (none) -> XDS100v2 Programmer:EEPROM_8pin
- Y1: footprint (none) -> Crystals:Crystal_SMD_HC49-SD
Changed lines of the file:
@@
 F 0 "J1" H 1407 2292 50  0000 C CNN
 F 1 "USB_B_Mini" H 1407 2201 50  0000 C CNN
-F 2 "" H 1500 1775 50  0001 C CNN
+F 2 "XDS100v2 Programmer:USB_Mini_B_32005-201" H 1500 1775 50  0001 C CNN
 F 3 "~" H 1500 1775 50  0001 C CNN
 F 4 "ED2992CT-ND" H 1350 1825 50  0001 C CNN "Digikey"
@@
 F 0 "F1" V 1678 1625 50  0000 C CNN
 F 1 "500mA" V 1769 1625 50  0000 C CNN
-F 2 "" V 1805 1625 50  0001 C CNN
+F 2 "XDS100v2 Programmer:1812_PloyFuse" V 1805 1625 50  0001 C CNN
 F 3 "~" H 1875 1625 50  0001 C CNN
 F 4 "MF-MSMF050-2CT-ND" V 1875 1625 50  0001 C CNN "Digikey"
@@
 F 0 "C4" H 3443 1896 50  0000 L CNN
 F 1 "100uF" H 3443 1805 50  0000 L CNN
-F 2 "" H 3363 1700 50  0001 C CNN
+F 2 "Capacitors_Tantalum_SMD:CP_Tantalum_Case-U_EIA-6032-15_Reflow" H 3363 1700 50  0001 C CNN
 F 3 "~" H 3325 1850 50  0001 C CNN
 F 4 "478-7995-1-ND" H 3325 1850 50  0001 C CNN "Digikey"
@@
 F 0 "Y1" V 4804 5088 50  0000 L CNN
 F 1 "12MHz" V 4895 5088 50  0000 L CNN
-F 2 "" H 4850 5000 50  0001 C CNN
+F 2 "Crystals:Crystal_SMD_HC49-SD" H 4850 5000 50  0001 C CNN
 F 3 "~" H 4850 5000 50  0001 C CNN
 F 4 "XC2079CT-ND" V 4850 5000 50  0001 C CNN "Digikey"
@@
 F 0 "SW1" H 8950 5067 50  0000 C CNN
 F 1 "SW_DIP_x02" H 8950 4976 50  0000 C CNN
-F 2 "" H 8950 4700 50  0001 C CNN
+F 2 "XDS100v2 Programmer:CTS_DPST_Switch" H 8950 4700 50  0001 C CNN
 F 3 "~" H 8950 4700 50  0001 C CNN
 F 4 "CT204211ST-ND" H 8950 4700 50  0001 C CNN "Digikey"
@@
 F 0 "SW2" H 8950 5642 50  0000 C CNN
 F 1 "SW_DIP_x02" H 8950 5551 50  0000 C CNN
-F 2 "" H 8950 5275 50  0001 C CNN
+F 2 "XDS100v2 Programmer:CTS_DPST_Switch" H 8950 5275 50  0001 C CNN
 F 3 "~" H 8950 5275 50  0001 C CNN
 F 4 "CT204211ST-ND" H 8950 5275 50  0001 C CNN "Digikey"
@@
 F 0 "SW3" H 8950 6417 50  0000 C CNN
 F 1 "SW_DIP_x03" H 8950 6326 50  0000 C CNN
-F 2 "" H 8950 5950 50  0001 C CNN
+F 2 "XDS100v2 Programmer:CTS_3DIP_Switch" H 8950 5950 50  0001 C CNN
 F 3 "~" H 8950 5950 50  0001 C CNN
 F 4 "CT2043ST-ND" H 8950 5950 50  0001 C CNN "Digikey"
@@
 F 0 "J2" H 10475 5000 50  0000 C CNN
 F 1 "Conn_02x05" H 10475 4400 50  0000 C CNN
-F 2 "" H 10425 4700 50  0001 C CNN
+F 2 "Pin_Headers:Pin_Header_Straight_2x05_Pitch2.54mm" H 10425 4700 50  0001 C CNN
 F 3 "~" H 10425 4700 50  0001 C CNN
 F 4 "ED1543-ND" H 10425 4700 50  0001 C CNN "Digikey"
@@
 F 0 "U6" H 2475 4815 50  0000 C CNN
 F 1 "EEPROM_Array_8pin" H 2475 4724 50  0000 C CNN
-F 2 "" H 2625 4400 50  0001 C CNN
+F 2 "XDS100v2 Programmer:EEPROM_8pin" H 2625 4400 50  0001 C CNN
 F 3 "" H 2625 4400 50  0001 C CNN
 F 4 "1662-2080-1-ND‎" H 2475 4400 50  0001 C CNN "Digikey"
@@
 $EndComp
 $Comp
-L Mechanical:MountingHole_Pad H?
+L Mechanical:MountingHole_Pad H1
 U 1 1 5EC57A13
 P 8425 775
-F 0 "H?" H 8525 778 50  0000 L CNN
+F 0 "H1" H 8525 778 50  0000 L CNN
 F 1 "MountingHole_Pad" H 8525 733 50  0001 L CNN
-F 2 "" H 8425 775 50  0001 C CNN
+F 2 "Mounting_Holes:MountingHole_3mm_Pad_Via" H 8425 775 50  0001 C CNN
 F 3 "~" H 8425 775 50  0001 C CNN
 	1    8425 775
@@
 $EndComp
 $Comp
-L Mechanical:MountingHole_Pad H?
+L Mechanical:MountingHole_Pad H2
 U 1 1 5EC59DEB
 P 8775 775
-F 0 "H?" H 8875 778 50  0000 L CNN
+F 0 "H2" H 8875 778 50  0000 L CNN
 F 1 "MountingHole_Pad" H 8875 733 50  0001 L CNN
-F 2 "" H 8775 775 50  0001 C CNN
+F 2 "Mounting_Holes:MountingHole_3mm_Pad_Via" H 8775 775 50  0001 C CNN
 F 3 "~" H 8775 775 50  0001 C CNN
 	1    8775 775
@@
 $EndComp
 $Comp
-L Mechanical:MountingHole_Pad H?
+L Mechanical:MountingHole_Pad H3
 U 1 1 5EC5A192
 P 9125 775
-F 0 "H?" H 9225 778 50  0000 L CNN
+F 0 "H3" H 9225 778 50  0000 L CNN
 F 1 "MountingHole_Pad" H 9225 733 50  0001 L CNN
-F 2 "" H 9125 775 50  0001 C CNN
+F 2 "Mounting_Holes:MountingHole_3mm_Pad_Via" H 9125 775 50  0001 C CNN
 F 3 "~" H 9125 775 50  0001 C CNN
 	1    9125 775
@@
 $EndComp
 $Comp
-L Mechanical:MountingHole_Pad H?
+L Mechanical:MountingHole_Pad H4
 U 1 1 5EC5A687
 P 9450 775
-F 0 "H?" H 9550 778 50  0000 L CNN
+F 0 "H4" H 9550 778 50  0000 L CNN
 F 1 "MountingHole_Pad" H 9550 733 50  0001 L CNN
-F 2 "" H 9450 775 50  0001 C CNN
+F 2 "Mounting_Holes:MountingHole_3mm_Pad_Via" H 9450 775 50  0001 C CNN
 F 3 "~" H 9450 775 50  0001 C CNN
 	1    9450 775
@@
 $EndComp
 $Comp
-L power:GNDD #PWR?
+L power:GNDD #PWR0149
 U 1 1 5EC5AED7
 P 8425 950
-F 0 "#PWR?" H 8425 700 50  0001 C CNN
+F 0 "#PWR0149" H 8425 700 50  0001 C CNN
 F 1 "GNDD" H 8429 795 50  0000 C CNN
 F 2 "" H 8425 950 50  0001 C CNN
@@
 	8425 875  8425 950
 $Comp
-L power:GNDD #PWR?
+L power:GNDD #PWR0150
 U 1 1 5EC6C740
 P 8775 950
-F 0 "#PWR?" H 8775 700 50  0001 C CNN
+F 0 "#PWR0150" H 8775 700 50  0001 C CNN
 F 1 "GNDD" H 8779 795 50  0000 C CNN
 F 2 "" H 8775 950 50  0001 C CNN
@@
 	8775 875  8775 950
 $Comp
-L power:GNDD #PWR?
+L power:GNDD #PWR0151
 U 1 1 5EC7D792
 P 9125 950
-F 0 "#PWR?" H 9125 700 50  0001 C CNN
+F 0 "#PWR0151" H 9125 700 50  0001 C CNN
 F 1 "GNDD" H 9129 795 50  0000 C CNN
 F 2 "" H 9125 950 50  0001 C CNN
@@
 	9125 875  9125 950
 $Comp
-L power:GNDD #PWR?
+L power:GNDD #PWR0152
 U 1 1 5EC8E96E
 P 9450 950
-F 0 "#PWR?" H 9450 700 50  0001 C CNN
+F 0 "#PWR0152" H 9450 700 50  0001 C CNN
 F 1 "GNDD" H 9454 795 50  0000 C CNN
 F 2 "" H 9450 950 50  0001 C CNN
@@
 	9450 875  9450 950
 $Comp
-L Mechanical:MountingHole_Pad H?
+L Mechanical:MountingHole_Pad H5
 U 1 1 5ECB6AC0
 P 10250 775
-F 0 "H?" H 10350 778 50  0000 L CNN
+F 0 "H5" H 10350 778 50  0000 L CNN
 F 1 "MountingHole_Pad" H 10350 733 50  0001 L CNN
-F 2 "" H 10250 775 50  0001 C CNN
+F 2 "Mounting_Holes:MountingHole_3mm_Pad_Via" H 10250 775 50  0001 C CNN
 F 3 "~" H 10250 775 50  0001 C CNN
 	1    10250 775
@@
 $EndComp
 $Comp
-L Mechanical:MountingHole_Pad H?
+L Mechanical:MountingHole_Pad H6
 U 1 1 5ECB6AC6
 P 10575 775
-F 0 "H?" H 10675 778 50  0000 L CNN
+F 0 "H6" H 10675 778 50  0000 L CNN
 F 1 "MountingHole_Pad" H 10675 733 50  0001 L CNN
-F 2 "" H 10575 775 50  0001 C CNN
+F 2 "Mounting_Holes:MountingHole_3mm_Pad_Via" H 10575 775 50  0001 C CNN
 F 3 "~" H 10575 775 50  0001 C CNN
 	1    10575 775
@@
 	10575 875  10575 950
 $Comp
-L power:GND #PWR?
+L power:GND #PWR0153
 U 1 1 5ECC751B
 P 10250 950
-F 0 "#PWR?" H 10250 700 50  0001 C CNN
+F 0 "#PWR0153" H 10250 700 50  0001 C CNN
 F 1 "GND" H 10255 777 50  0000 C CNN
 F 2 "" H 10250 950 50  0001 C CNN
@@
 $EndComp
 $Comp
-L power:GND #PWR?
+L power:GND #PWR0154
 U 1 1 5ECC7B09
 P 10575 950
-F 0 "#PWR?" H 10575 700 50  0001 C CNN
+F 0 "#PWR0154" H 10575 700 50  0001 C CNN
 F 1 "GND" H 10580 777 50  0000 C CNN
 F 2 "" H 10575 950 50  0001 C CNN

Commit message: Schematic Update
- Fixed small schematic issues (resistors in the wrong place)
- Add thermal pad to FTDI chip symbol
Parts:
- removed R1: 1k, Resistors_SMD:R_0805, symbol Device:R_Small_US
- added R?: 820, Resistors_SMD:R_0805, symbol Device:R_Small_US
- U4: symbol Interface_USB:FT2232H -> XDS100v2~Programmer:FT2232H
Connections:
- net labels removed: ~PWREN~, ~SUSPEND~
- no-connect marks 25 -> 27
Other:
- note added: "Boot Mode"
- note added: "PWR_ISO"
- note added: "Programming Cable \n Interface"
- note added: "XDS100 Serial"
- moved on the sheet: R3, R6
Changed lines of the file:
@@
 $EndComp
 $Comp
-L Interface_USB:FT2232H U4
+L XDS100v2~Programmer:FT2232H U4
 U 1 1 5E1F5D22
 P 6300 3600
@@
 L Device:R_Small_US R6
 U 1 1 5E2192E6
-P 4900 3200
-F 0 "R6" V 4825 3250 50  0000 L CNN
-F 1 "12k" V 4825 3000 50  0000 L CNN
-F 2 "Resistors_SMD:R_0805" H 4900 3200 50  0001 C CNN
-F 3 "~" H 4900 3200 50  0001 C CNN
-F 4 "A129762CT-ND" V 4900 3200 50  0001 C CNN "Digikey"
-	1    4900 3200
+P 4900 3300
+F 0 "R6" V 4825 3350 50  0000 L CNN
+F 1 "12k" V 4825 3100 50  0000 L CNN
+F 2 "Resistors_SMD:R_0805" H 4900 3300 50  0001 C CNN
+F 3 "~" H 4900 3300 50  0001 C CNN
+F 4 "A129762CT-ND" V 4900 3300 50  0001 C CNN "Digikey"
+	1    4900 3300
 	0    -1   -1   0
 $EndComp
@@
 L power:GNDD #PWR0111
 U 1 1 5E21BD98
-P 4450 3250
-F 0 "#PWR0111" H 4450 3000 50  0001 C CNN
-F 1 "GNDD" H 4454 3095 50  0000 C CNN
-F 2 "" H 4450 3250 50  0001 C CNN
-F 3 "" H 4450 3250 50  0001 C CNN
-	1    4450 3250
-	1    0    0    -1
-$EndComp
-$Comp
-L Device:R_Small_US R3
-U 1 1 5E220ADC
-P 4900 3000
-F 0 "R3" V 4825 3050 50  0000 L CNN
-F 1 "1k" V 4825 2850 50  0000 L CNN
-F 2 "Resistors_SMD:R_0805" H 4900 3000 50  0001 C CNN
-F 3 "~" H 4900 3000 50  0001 C CNN
-F 4 "311-1.0KARCT-ND" V 4900 3000 50  0001 C CNN "Digikey"
-	1    4900 3000
-	0    -1   -1   0
-$EndComp
-Wire Wire Line
-	5000 3000 5100 3000
-Wire Wire Line
-	5000 3200 5100 3200
+P 4625 3550
+F 0 "#PWR0111" H 4625 3300 50  0001 C CNN
+F 1 "GNDD" H 4629 3395 50  0000 C CNN
+F 2 "" H 4625 3550 50  0001 C CNN
+F 3 "" H 4625 3550 50  0001 C CNN
+	1    4625 3550
+	1    0    0    -1
+$EndComp
+Wire Wire Line
+	5000 3100 5100 3100
+Wire Wire Line
+	5000 3300 5100 3300
 $Comp
 L power:+3V3 #PWR0112
 U 1 1 5E225768
-P 4575 3150
-F 0 "#PWR0112" H 4575 3000 50  0001 C CNN
-F 1 "+3V3" H 4675 3150 50  0000 C CNN
-F 2 "" H 4575 3150 50  0001 C CNN
-F 3 "" H 4575 3150 50  0001 C CNN
-	1    4575 3150
+P 4625 3050
+F 0 "#PWR0112" H 4625 2900 50  0001 C CNN
+F 1 "+3V3" H 4625 3200 50  0000 C CNN
+F 2 "" H 4625 3050 50  0001 C CNN
+F 3 "" H 4625 3050 50  0001 C CNN
+	1    4625 3050
 	1    0    0    -1
 $EndComp
@@
 D-
 Wire Wire Line
-	4800 3200 4575 3200
-Wire Wire Line
-	4575 3200 4575 3150
-Wire Wire Line
-	4800 3000 4450 3000
-Wire Wire Line
-	4450 3000 4450 3250
+	4625 3100 4625 3050
+Wire Wire Line
+	4800 3300 4625 3300
+Wire Wire Line
+	4625 3300 4625 3550
 Wire Wire Line
 	5100 1700 4950 1700
@@
 NoConn ~ 7500 5000
 NoConn ~ 7500 5100
-Wire Wire Line
-	7500 5400 7900 5400
-Wire Wire Line
-	7500 5300 7900 5300
-Text Label 7900 5300 2    50   ~ 0
-~PWREN~
-Text Label 7900 5400 2    50   ~ 0
-~SUSPEND~
 $Comp
 L Device:LED D1
@@
 	0    -1   -1   0
 $EndComp
-$Comp
-L Device:R_Small_US R1
-U 1 1 5E2CDD04
-P 4125 1025
-F 0 "R1" H 4175 1100 50  0000 L CNN
-F 1 "1k" H 4175 975 50  0000 L CNN
-F 2 "Resistors_SMD:R_0805" H 4125 1025 50  0001 C CNN
-F 3 "~" H 4125 1025 50  0001 C CNN
-F 4 "311-1.0KARCT-ND" V 4125 1025 50  0001 C CNN "Digikey"
-	1    4125 1025
-	1    0    0    -1
-$EndComp
 Wire Wire Line
 	4125 1125 4125 1175
@@
 U 1 1 5EB64DD5
 P 1950 4400
-F 0 "C11" H 2100 4325 50  0000 R CNN
+F 0 "C11" H 2125 4325 50  0000 R CNN
 F 1 "0.1uF" H 2200 4475 50  0000 R CNN
 F 2 "Capacitors_SMD:C_0805" H 1950 4400 50  0001 C CNN
@@
 	1    0    0    -1
 $EndComp
+Wire Wire Line
+	4800 3100 4625 3100
+$Comp
+L Device:R_Small_US R3
+U 1 1 5E220ADC
+P 4900 3100
+F 0 "R3" V 4825 3150 50  0000 L CNN
+F 1 "1k" V 4825 2950 50  0000 L CNN
+F 2 "Resistors_SMD:R_0805" H 4900 3100 50  0001 C CNN
+F 3 "~" H 4900 3100 50  0001 C CNN
+F 4 "311-1.0KARCT-ND" V 4900 3100 50  0001 C CNN "Digikey"
+	1    4900 3100
+	0    -1   -1   0
+$EndComp
+Wire Wire Line
+	5500 5750 5500 6025
+Wire Wire Line
+	5500 6025 5700 6025
+Connection ~ 5700 6025
+$Comp
+L Device:R_Small_US R?
+U 1 1 5ED7B567
+P 4125 1025
+F 0 "R?" H 4175 1100 50  0000 L CNN
+F 1 "820" H 4175 975 50  0000 L CNN
+F 2 "Resistors_SMD:R_0805" H 4125 1025 50  0001 C CNN
+F 3 "~" H 4125 1025 50  0001 C CNN
+F 4 "311-820ARCT-ND" V 4125 1025 50  0001 C CNN "Digikey"
+	1    4125 1025
+	1    0    0    -1
+$EndComp
+NoConn ~ 7500 5300
+NoConn ~ 7500 5400
+Text Notes 9250 4475 0    50   ~ 0
+PWR_ISO
+Text Notes 9625 5250 0    50   ~ 0
+XDS100 Serial
+Text Notes 8250 5600 0    50   ~ 0
+Boot Mode
+Text Notes 10125 4375 0    50   ~ 0
+Programming Cable \n     Interface
 $EndSCHEMATC

Commit message: Netlist & PCB
- Created netlist
- Initial layout import
Parts:
- gave numbers to parts that had none: 1
Changed lines of the file:
@@
 Connection ~ 5700 6025
 $Comp
-L Device:R_Small_US R?
+L Device:R_Small_US R1
 U 1 1 5ED7B567
 P 4125 1025
-F 0 "R?" H 4175 1100 50  0000 L CNN
+F 0 "R1" H 4175 1100 50  0000 L CNN
 F 1 "820" H 4175 975 50  0000 L CNN
 F 2 "Resistors_SMD:R_0805" H 4125 1025 50  0001 C CNN

Commit message: Changed Output Pinout
- Changed programming cable connector to follow ARM 10 Pin JTAG standard, although it is slightly modified.
Parts:
- removed J2: Conn_02x05, Pin_Headers:Pin_Header_Straight_2x05_Pitch2.54mm, symbol Connector_Generic:Conn_02x05_Counter_Clockwise
- added J?: Conn_02x05_Odd_Even, symbol Connector_Generic:Conn_02x05_Odd_Even
Other:
- note added: "Follows ARM 10 Pin JTAG Interface, \nslightly modified"
Changed lines of the file:
@@
 Text Label 8350 5275 0    50   ~ 0
 SCI_TX
-Text Label 10975 4800 2    50   ~ 0
+Text Label 10975 4700 2    50   ~ 0
 TDO
 Text Label 9850 4500 0    50   ~ 0
@@
 Text Label 8350 5175 0    50   ~ 0
 SCI_RX
-Text Label 10975 4700 2    50   ~ 0
+Text Label 10975 4500 2    50   ~ 0
 TMS
+Text Label 10975 4800 2    50   ~ 0
+TDI
 Text Label 10975 4600 2    50   ~ 0
-TDI
-Text Label 10975 4900 2    50   ~ 0
 TCK
 $Comp
@@
 Wire Wire Line
 	8125 5750 8650 5750
-Text Label 10975 4500 2    50   ~ 0
+Text Label 10975 4900 2    50   ~ 0
 TRST
 Text Label 9850 4800 0    50   ~ 0
@@
 Text Label 9850 4700 0    50   ~ 0
 GPIO29
-$Comp
-L Connector_Generic:Conn_02x05_Counter_Clockwise J2
-U 1 1 5EA078BB
-P 10425 4700
-F 0 "J2" H 10475 5000 50  0000 C CNN
-F 1 "Conn_02x05" H 10475 4400 50  0000 C CNN
-F 2 "Pin_Headers:Pin_Header_Straight_2x05_Pitch2.54mm" H 10425 4700 50  0001 C CNN
-F 3 "~" H 10425 4700 50  0001 C CNN
-F 4 "ED1543-ND" H 10425 4700 50  0001 C CNN "Digikey"
-	1    10425 4700
-	1    0    0    -1
-$EndComp
 Wire Wire Line
 	10975 4500 10725 4500
@@
 Text Notes 9250 4475 0    50   ~ 0
 PWR_ISO
-Text Notes 9625 5250 0    50   ~ 0
+Text Notes 7725 5225 0    50   ~ 0
 XDS100 Serial
 Text Notes 8250 5600 0    50   ~ 0
 Boot Mode
-Text Notes 10125 4375 0    50   ~ 0
+Text Notes 10125 4325 0    50   ~ 0
 Programming Cable \n     Interface
+Text Notes 10150 5125 0    39   Italic 0
+Follows ARM 10 Pin JTAG Interface, \nslightly modified
+$Comp
+L Connector_Generic:Conn_02x05_Odd_Even J?
+U 1 1 5E219B1D
+P 10425 4700
+F 0 "J?" H 10475 5000 50  0000 C CNN
+F 1 "Conn_02x05_Odd_Even" H 10500 4400 50  0001 C CNN
+F 2 "" H 10425 4700 50  0001 C CNN
+F 3 "~" H 10425 4700 50  0001 C CNN
+	1    10425 4700
+	1    0    0    -1
+$EndComp
 $EndSCHEMATC

Commit message: Removed Pulldown
- Removed pulldown on TRST line
- Will be permanently added to the main test board or integrated board.
- If programmer is not plugged in, the board will automatically boot to flash. If connected, the option is there to connect the TRST pin to JTAGTRST for JTAG debugging, while still enabling boot from flash.
Parts:
- removed R15: 2.2k, Resistors_SMD:R_0805, symbol Device:R_Small_US
Connections:
- wire segments 266 -> 263
Changed lines of the file:
@@
 	9600 5400 9975 5400
 Connection ~ 9600 5400
-Wire Wire Line
-	8650 5950 8600 5950
 Text Label 7825 5750 0    50   ~ 0
 GPIO34
@@
 Wire Wire Line
 	8375 5850 7825 5850
-Wire Wire Line
-	8600 5950 8600 6025
 $Comp
 L Device:R_Small_US R13
@@
 Wire Wire Line
 	8375 6300 8375 6225
-$Comp
-L power:GND #PWR0145
-U 1 1 5E8FAD6F
-P 8600 6300
-F 0 "#PWR0145" H 8600 6050 50  0001 C CNN
-F 1 "GND" H 8605 6127 50  0000 C CNN
-F 2 "" H 8600 6300 50  0001 C CNN
-F 3 "" H 8600 6300 50  0001 C CNN
-	1    8600 6300
-	1    0    0    -1
-$EndComp
-Wire Wire Line
-	8600 6300 8600 6225
-Wire Wire Line
-	7825 5950 8600 5950
-Connection ~ 8600 5950
 Wire Wire Line
 	8375 5850 8650 5850
@@
 F 4 "311-2.20KCRCT-ND" V 8375 6125 50  0001 C CNN "Digikey"
 	1    8375 6125
-	1    0    0    -1
-$EndComp
-$Comp
-L Device:R_Small_US R15
-U 1 1 5EAF1D16
-P 8600 6125
-F 0 "R15" H 8500 6225 50  0000 L CNN
-F 1 "2.2k" H 8400 6075 50  0000 L CNN
-F 2 "Resistors_SMD:R_0805" H 8600 6125 50  0001 C CNN
-F 3 "~" H 8600 6125 50  0001 C CNN
-F 4 "311-2.20KCRCT-ND" V 8600 6125 50  0001 C CNN "Digikey"
-	1    8600 6125
 	1    0    0    -1
 $EndComp
@@
 	1    0    0    -1
 $EndComp
+Wire Wire Line
+	7825 5950 8650 5950
 $EndSCHEMATC

Commit message: Removed Unused Pins
- GPIO34 and TDO switch options are useless for this application, removed them to reduce complexity.
- Updated programming pin interface
Parts:
- removed R11, R12: 820, Resistors_SMD:R_0805, symbol Device:R_Small_US
- removed R13, R14: 2.2k, Resistors_SMD:R_0805, symbol Device:R_Small_US
Connections:
- net labels removed: GPIO34
- wire segments 263 -> 249
- no-connect marks 27 -> 31
Changed lines of the file:
@@
 	1    0    0    -1
 $EndComp
-Text Label 9650 5950 2    50   ~ 0
+Text Label 9700 5950 2    50   ~ 0
 JTAG_TRST
 Wire Wire Line
-	9250 5950 9650 5950
-$Comp
-L Device:R_Small_US R11
-U 1 1 5E78A36F
-P 9350 5625
-F 0 "R11" H 9400 5700 50  0000 L CNN
-F 1 "820" H 9400 5575 50  0000 L CNN
-F 2 "Resistors_SMD:R_0805" H 9350 5625 50  0001 C CNN
-F 3 "~" H 9350 5625 50  0001 C CNN
-F 4 "311-820ARCT-ND" V 9350 5625 50  0001 C CNN "Digikey"
-	1    9350 5625
-	1    0    0    -1
-$EndComp
-Wire Wire Line
-	9250 5750 9350 5750
-Wire Wire Line
-	9350 5750 9350 5725
-Wire Wire Line
-	9250 5850 9600 5850
-Wire Wire Line
-	9600 5725 9600 5850
-$Comp
-L Device:R_Small_US R12
-U 1 1 5E7ACE17
-P 9600 5625
-F 0 "R12" H 9650 5700 50  0000 L CNN
-F 1 "820" H 9650 5575 50  0000 L CNN
-F 2 "Resistors_SMD:R_0805" H 9600 5625 50  0001 C CNN
-F 3 "~" H 9600 5625 50  0001 C CNN
-F 4 "311-820ARCT-ND" V 9600 5625 50  0001 C CNN "Digikey"
-	1    9600 5625
-	1    0    0    -1
-$EndComp
-Text Label 9975 5400 2    50   ~ 0
-3V3_MCU
-Wire Wire Line
-	9350 5400 9350 5525
-Wire Wire Line
-	9600 5400 9600 5525
-Wire Wire Line
-	9350 5400 9600 5400
-Wire Wire Line
-	9600 5400 9975 5400
-Connection ~ 9600 5400
-Text Label 7825 5750 0    50   ~ 0
-GPIO34
-Text Label 7825 5850 0    50   ~ 0
-TDO
-Text Label 7825 5950 0    50   ~ 0
+	9250 5950 9700 5950
+Text Label 8300 5950 0    50   ~ 0
 TRST
-Wire Wire Line
-	8125 5750 8125 6025
-Wire Wire Line
-	8375 5850 8375 6025
-Connection ~ 8375 5850
-Wire Wire Line
-	8375 5850 7825 5850
-$Comp
-L Device:R_Small_US R13
-U 1 1 5E865275
-P 8125 6125
-F 0 "R13" H 8025 6225 50  0000 L CNN
-F 1 "2.2k" H 7925 6075 50  0000 L CNN
-F 2 "Resistors_SMD:R_0805" H 8125 6125 50  0001 C CNN
-F 3 "~" H 8125 6125 50  0001 C CNN
-F 4 "311-2.20KCRCT-ND" V 8125 6125 50  0001 C CNN "Digikey"
-	1    8125 6125
-	1    0    0    -1
-$EndComp
-Connection ~ 8125 5750
-Wire Wire Line
-	8125 5750 7825 5750
-Wire Wire Line
-	8125 6225 8125 6300
-$Comp
-L power:GND #PWR0143
-U 1 1 5E8E1446
-P 8125 6300
-F 0 "#PWR0143" H 8125 6050 50  0001 C CNN
-F 1 "GND" H 8130 6127 50  0000 C CNN
-F 2 "" H 8125 6300 50  0001 C CNN
-F 3 "" H 8125 6300 50  0001 C CNN
-	1    8125 6300
-	1    0    0    -1
-$EndComp
-$Comp
-L power:GND #PWR0144
-U 1 1 5E8EDF4D
-P 8375 6300
-F 0 "#PWR0144" H 8375 6050 50  0001 C CNN
-F 1 "GND" H 8380 6127 50  0000 C CNN
-F 2 "" H 8375 6300 50  0001 C CNN
-F 3 "" H 8375 6300 50  0001 C CNN
-	1    8375 6300
-	1    0    0    -1
-$EndComp
-Wire Wire Line
-	8375 6300 8375 6225
-Wire Wire Line
-	8375 5850 8650 5850
-Wire Wire Line
-	8125 5750 8650 5750
 Text Label 10975 4900 2    50   ~ 0
 TRST
-Text Label 9850 4800 0    50   ~ 0
-GPIO34
 Text Label 9850 4600 0    50   ~ 0
 GPIO28
@@
 	9850 4700 10225 4700
 Wire Wire Line
-	9850 4800 10225 4800
-Wire Wire Line
 	10000 4925 10000 4900
 Wire Wire Line
-	10000 4900 10225 4900
-$Comp
-L Device:R_Small_US R14
-U 1 1 5EAF18B3
-P 8375 6125
-F 0 "R14" H 8275 6225 50  0000 L CNN
-F 1 "2.2k" H 8175 6075 50  0000 L CNN
-F 2 "Resistors_SMD:R_0805" H 8375 6125 50  0001 C CNN
-F 3 "~" H 8375 6125 50  0001 C CNN
-F 4 "311-2.20KCRCT-ND" V 8375 6125 50  0001 C CNN "Digikey"
-	1    8375 6125
-	1    0    0    -1
-$EndComp
+	10000 4900 10150 4900
 $Comp
 L XDS100v2~Programmer:EEPROM_Array_8pin U6
@@
 $EndComp
 Wire Wire Line
-	7825 5950 8650 5950
+	8300 5950 8650 5950
+Wire Wire Line
+	10225 4800 10150 4800
+Wire Wire Line
+	10150 4800 10150 4900
+Connection ~ 10150 4900
+Wire Wire Line
+	10150 4900 10225 4900
+NoConn ~ 9250 5850
+NoConn ~ 9250 5750
+NoConn ~ 8650 5750
+NoConn ~ 8650 5850
 $EndSCHEMATC
