File: PCBs/XDS100v2 Programmer/XDS100v2 Programmer.kicad_pcb (KiCad board)
At the start: 2 copper layers, 91 x 38 mm, 43 parts, among them J1 USB_B_Mini, J2 Conn_02x05_Odd_Even, SW1 SW_DIP_x02, SW2 SW_DIP_x02, SW3 SW_DIP_x03, U1 TLV1117-33, U2 ISO7240, U3 EEPROM_Array, U4 FT2232H, U5 ISO7231, U6 EEPROM_Array_8pin, Y1 12MHz

Commit message: Silkscreen
- Updated silkscreen
Parts:
- moved D2 1.90 mm to (60.5, 67.8)
Routing:
- net /D+: track 46.6 -> 44.9 mm, vias 2 -> 0
- net /D-: track 46.8 -> 45.1 mm, vias 2 -> 0
- net Net-(D2-Pad1): track 4.10 -> 5.31 mm
- net +3V3: track 191.1 -> 191.6 mm, vias 15 -> 17
Other:
- board text added: "+3V3"
- board text added: "BOOT"
- board text added: "For TI TMS320F MCUs"
- board text added: "Mark Belbin -- 2020"
- board text added: "New EEPROM"
- board text added: "Old EEPROM"
- board text added: "RX"
- board text added: "TX"
- board text added: "UART"
- board text added: "USB_PWR"
- board text added: "XDS100v2 Programmer"
