File: PCBs/MCU_Powertrain/MCU_Powertrain.sch (KiCad schematic (older format))
At the start: 0 parts

Commit message: Schematic Changes
- Added TI MCU Symbol
- Added Powertrain V1 schematic
- Setup Hierarcical Sheets
Other:
- note added: "CAN"
- note added: "Phases"
- note added: "Power Input"
- note added: "Powertrain"
- note added: "Programming"
- note added: "TI MCU"
Changed lines of the file:
@@
 $Descr A4 11693 8268
 encoding utf-8
-Sheet 1 1
+Sheet 1 3
 Title "MCU and Powertrain Test PCB"
 Date "2020-01-15"
@@
 Comment4 ""
 $EndDescr
+$Sheet
+S 7100 2625 2650 1700
+U 5E20A2BB
+F0 "Powertrain" 50
+F1 "Powertrain.sch" 50
+$EndSheet
+$Sheet
+S 3425 2625 2675 1700
+U 5E20A372
+F0 "TI_MCU" 50
+F1 "TI_MCU.sch" 50
+$EndSheet
+Text Notes 4375 3550 0    118  Italic 24
+TI MCU
+Text Notes 7950 3525 0    118  Italic 24
+Powertrain
+Text Notes 1075 1125 0    118  Italic 24
+Power Input
+Text Notes 1075 3600 0    118  Italic 24
+Programming
+Text Notes 4475 5350 0    118  Italic 24
+CAN
+Text Notes 10200 2625 0    118  Italic 24
+Phases
 $EndSCHEMATC

Commit message: More Schematic Changes
- Connected TI_MCU schematic to Powertrain schematic
- Added power input
Parts:
- added C?: 0.1uF, Capacitors_SMD:C_0603, symbol Device:C_Small
- added C?: 0.33uF, Capacitors_SMD:C_0603, symbol Device:C_Small
- added C?: 22uF, Capacitors_SMD:C_0805, symbol Device:C_Small
- added D?: D_Schottky_ALT, Diodes_SMD:D_SOD-123F, symbol Device:D_Schottky_ALT
- added D?: GREEN, LEDs:LED_0603, symbol Device:LED_ALT
- added J?: PWRIN, symbol Connector_Generic:Conn_01x02
- added J?: PHASE_A, ESC Drivetrain V1:3mm_Bullet_A, symbol Connector_Generic:Conn_01x01
- added J?: PHASE_B, ESC Drivetrain V1:3mm_Bullet_B, symbol Connector_Generic:Conn_01x01
- added J?: PHASE_C, ESC Drivetrain V1:3mm_Bullet_C, symbol Connector_Generic:Conn_01x01
- added J?: Big Conn, symbol Connector_Generic:Conn_02x05_Odd_Even
- added J?: Pogo Conn, symbol Connector_Generic:Conn_02x05_Odd_Even
- added L?: 15uH, ESC Drivetrain V1:Eaton_Inductor, symbol Device:L_Core_Ferrite
- added R?: 68.0kΩ, Resistors_SMD:R_0603, symbol Device:R_US
- added R?: 20.0kΩ, Resistors_SMD:R_0603, symbol Device:R_US
- added R?: 330Ω, Resistors_SMD:R_0603, symbol Device:R_US
- added U?: LMR16006XDDC, TO_SOT_Packages_SMD:SOT-23-6, symbol ESC~Drivetrain~V1:LMR16006XDDC
Connections:
- net labels added: +3V3, +BATT, GND
- wire segments 0 -> 59
- no-connect marks 0 -> 1
Other:
- note added: "3.3V Regulator"
- note added: "Up to 24V"

Commit message: Added Programming Headers
- Inserted programming headers based on latest header format from custom XDS100v2 programmer.
Parts:
- removed J?: Pogo Conn, symbol Connector_Generic:Conn_02x05_Odd_Even
- added J?: Pogo Conn, symbol Connector_Generic:Conn_02x05_Odd_Even
Connections:
- net labels added: GPIO28, GPIO29, TCK, TDI, TDO, TMS, TRST
- wire segments 59 -> 104
Changed lines of the file:
@@
 F21 "GPIO6" O R 6375 2925 50
 F22 "GPIO7" O R 6375 2850 50
-F23 "GPIO29" I L 3425 3350 50
-F24 "GPIO34" I L 3425 3250 50
-F25 "TRST" I L 3425 3450 50
-F26 "TCK" I L 3425 3550 50
-F27 "TMS" I L 3425 3650 50
-F28 "TDI" I L 3425 3750 50
-F29 "TDO" I L 3425 3850 50
+F23 "GPIO29" I L 3425 3225 50
+F24 "TRST" I L 3425 3850 50
+F25 "TCK" I L 3425 3550 50
+F26 "TMS" I L 3425 3450 50
+F27 "TDI" I L 3425 3750 50
+F28 "TDO" I L 3425 3650 50
+F29 "GPIO28" I L 3425 3125 50
 $EndSheet
 Text Notes 4375 3550 0    118  Italic 24
@@
 	1    0    0    -1
 $EndComp
+Wire Wire Line
+	6375 2700 7100 2700
+Wire Wire Line
+	7100 2775 6375 2775
+Wire Wire Line
+	6375 2850 7100 2850
+Wire Wire Line
+	7100 2925 6375 2925
+Wire Wire Line
+	6375 3050 7100 3050
+Wire Wire Line
+	7100 3125 6375 3125
+Wire Wire Line
+	6375 3200 7100 3200
+Wire Wire Line
+	7100 3275 6375 3275
+Wire Wire Line
+	6375 3350 7100 3350
+Wire Wire Line
+	7100 3425 6375 3425
+Wire Wire Line
+	6375 3500 7100 3500
+Wire Wire Line
+	7100 3625 6375 3625
+Wire Wire Line
+	6375 3700 7100 3700
+Wire Wire Line
+	7100 3775 6375 3775
+Wire Wire Line
+	6375 3850 7100 3850
+Wire Wire Line
+	7100 3925 6375 3925
+Wire Wire Line
+	6375 4000 7100 4000
+Wire Wire Line
+	7100 4175 6375 4175
+Wire Wire Line
+	6375 4250 7100 4250
+Wire Wire Line
+	7100 4325 6375 4325
+Wire Wire Line
+	6375 4400 7100 4400
+Wire Wire Line
+	1075 3675 875  3675
+Wire Wire Line
+	875  3675 875  3600
+Wire Wire Line
+	1075 3975 1000 3975
+Wire Wire Line
+	1000 3975 1000 4075
+Wire Wire Line
+	1075 4075 1000 4075
+Wire Wire Line
+	1000 4075 875  4075
+Wire Wire Line
+	875  4075 875  4125
+Connection ~ 1000 4075
+$Comp
+L power:GND #PWR?
+U 1 1 5E266250
+P 875 4125
+AR Path="/5E20A2BB/5E266250" Ref="#PWR?"  Part="1"
+AR Path="/5E266250" Ref="#PWR?"  Part="1"
+F 0 "#PWR?" H 875 3875 50  0001 C CNN
+F 1 "GND" H 880 3952 50  0000 C CNN
+F 2 "" H 875 4125 50  0001 C CNN
+F 3 "" H 875 4125 50  0001 C CNN
+	1    875  4125
+	1    0    0    -1
+$EndComp
+$Comp
+L power:+3V3 #PWR?
+U 1 1 5E266D11
+P 875 3600
+AR Path="/5E20A2BB/5E266D11" Ref="#PWR?"  Part="1"
+AR Path="/5E266D11" Ref="#PWR?"  Part="1"
+F 0 "#PWR?" H 875 3450 50  0001 C CNN
+F 1 "+3V3" H 1025 3675 50  0000 C CNN
+F 2 "" H 875 3600 50  0001 C CNN
+F 3 "" H 875 3600 50  0001 C CNN
+	1    875  3600
+	1    0    0    -1
+$EndComp
+Text Label 800  3775 0    50   ~ 0
+GPIO28
+Wire Wire Line
+	800  3775 1075 3775
+Wire Wire Line
+	800  3875 1075 3875
+Text Label 800  3875 0    50   ~ 0
+GPIO29
+Text Label 1825 3675 2    50   ~ 0
+TMS
+Text Label 1825 3775 2    50   ~ 0
+TCK
+Text Label 1825 3875 2    50   ~ 0
+TDO
+Text Label 1825 3975 2    50   ~ 0
+TDI
+Text Label 1825 4075 2    50   ~ 0
+TRST
 $Comp
 L Connector_Generic:Conn_02x05_Odd_Even J?
-U 1 1 5E5BBE7F
-P 1275 4600
-F 0 "J?" H 1325 4925 50  0000 C CNN
-F 1 "Pogo Conn" H 1325 4275 50  0000 C CNN
-F 2 "" H 1275 4600 50  0001 C CNN
-F 3 "~" H 1275 4600 50  0001 C CNN
-	1    1275 4600
-	1    0    0    -1
-$EndComp
-Wire Wire Line
-	6375 2700 7100 2700
-Wire Wire Line
-	7100 2775 6375 2775
-Wire Wire Line
-	6375 2850 7100 2850
-Wire Wire Line
-	7100 2925 6375 2925
-Wire Wire Line
-	6375 3050 7100 3050
-Wire Wire Line
-	7100 3125 6375 3125
-Wire Wire Line
-	6375 3200 7100 3200
-Wire Wire Line
-	7100 3275 6375 3275
-Wire Wire Line
-	6375 3350 7100 3350
-Wire Wire Line
-	7100 3425 6375 3425
-Wire Wire Line
-	6375 3500 7100 3500
-Wire Wire Line
-	7100 3625 6375 3625
-Wire Wire Line
-	6375 3700 7100 3700
-Wire Wire Line
-	7100 3775 6375 3775
-Wire Wire Line
-	6375 3850 7100 3850
-Wire Wire Line
-	7100 3925 6375 3925
-Wire Wire Line
-	6375 4000 7100 4000
-Wire Wire Line
-	7100 4175 6375 4175
-Wire Wire Line
-	6375 4250 7100 4250
-Wire Wire Line
-	7100 4325 6375 4325
-Wire Wire Line
-	6375 4400 7100 4400
+U 1 1 5E2798B5
+P 1275 4800
+F 0 "J?" H 1325 5125 50  0000 C CNN
+F 1 "Pogo Conn" H 1325 4475 50  0000 C CNN
+F 2 "" H 1275 4800 50  0001 C CNN
+F 3 "~" H 1275 4800 50  0001 C CNN
+	1    1275 4800
+	1    0    0    -1
+$EndComp
+Wire Wire Line
+	1075 4600 875  4600
+Wire Wire Line
+	875  4600 875  4525
+Wire Wire Line
+	1075 4900 1000 4900
+Wire Wire Line
+	1000 4900 1000 5000
+Wire Wire Line
+	1075 5000 1000 5000
+Wire Wire Line
+	1000 5000 875  5000
+Wire Wire Line
+	875  5000 875  5050
+Connection ~ 1000 5000
+$Comp
+L power:GND #PWR?
+U 1 1 5E2798C3
+P 875 5050
+AR Path="/5E20A2BB/5E2798C3" Ref="#PWR?"  Part="1"
+AR Path="/5E2798C3" Ref="#PWR?"  Part="1"
+F 0 "#PWR?" H 875 4800 50  0001 C CNN
+F 1 "GND" H 880 4877 50  0000 C CNN
+F 2 "" H 875 5050 50  0001 C CNN
+F 3 "" H 875 5050 50  0001 C CNN
+	1    875  5050
+	1    0    0    -1
+$EndComp
+$Comp
+L power:+3V3 #PWR?
+U 1 1 5E2798C9
+P 875 4525
+AR Path="/5E20A2BB/5E2798C9" Ref="#PWR?"  Part="1"
+AR Path="/5E2798C9" Ref="#PWR?"  Part="1"
+F 0 "#PWR?" H 875 4375 50  0001 C CNN
+F 1 "+3V3" H 1025 4600 50  0000 C CNN
+F 2 "" H 875 4525 50  0001 C CNN
+F 3 "" H 875 4525 50  0001 C CNN
+	1    875  4525
+	1    0    0    -1
+$EndComp
+Text Label 800  4700 0    50   ~ 0
+GPIO28
+Wire Wire Line
+	800  4700 1075 4700
+Wire Wire Line
+	800  4800 1075 4800
+Text Label 800  4800 0    50   ~ 0
+GPIO29
+Text Label 1825 4600 2    50   ~ 0
+TMS
+Text Label 1825 4700 2    50   ~ 0
+TCK
+Text Label 1825 4800 2    50   ~ 0
+TDO
+Text Label 1825 4900 2    50   ~ 0
+TDI
+Text Label 1825 5000 2    50   ~ 0
+TRST
+Wire Wire Line
+	3425 3225 3100 3225
+Wire Wire Line
+	3425 3125 3100 3125
+Text Label 3100 3125 0    50   ~ 0
+GPIO28
+Text Label 3100 3225 0    50   ~ 0
+GPIO29
+Wire Wire Line
+	2275 3450 2275 3675
+Wire Wire Line
+	1575 3675 2275 3675
+Wire Wire Line
+	2275 3450 3425 3450
+Wire Wire Line
+	2350 3550 2350 3775
+Wire Wire Line
+	1575 3775 2350 3775
+Wire Wire Line
+	2350 3550 3425 3550
+Wire Wire Line
+	2425 3650 2425 3875
+Wire Wire Line
+	1575 3875 2425 3875
+Wire Wire Line
+	2425 3650 3425 3650
+Wire Wire Line
+	2500 3750 2500 3975
+Wire Wire Line
+	1575 3975 2500 3975
+Wire Wire Line
+	2500 3750 3425 3750
+Wire Wire Line
+	2575 3850 2575 4075
+Wire Wire Line
+	1575 4075 2575 4075
+Wire Wire Line
+	2575 3850 3425 3850
+Wire Wire Line
+	2275 3675 2275 4600
+Wire Wire Line
+	1575 4600 2275 4600
+Connection ~ 2275 3675
+Wire Wire Line
+	2350 3775 2350 4700
+Wire Wire Line
+	1575 4700 2350 4700
+Connection ~ 2350 3775
+Wire Wire Line
+	2425 3875 2425 4800
+Wire Wire Line
+	1575 4800 2425 4800
+Connection ~ 2425 3875
+Wire Wire Line
+	2500 3975 2500 4900
+Wire Wire Line
+	1575 4900 2500 4900
+Connection ~ 2500 3975
+Wire Wire Line
+	2575 4075 2575 5000
+Wire Wire Line
+	1575 5000 2575 5000
+Connection ~ 2575 4075
 $EndSCHEMATC

Commit message: CAN and Minor Changes
- Added CAN Controller (MCP2515) and CAN transciever
- Added net-ties to shunts
- Removed all +12V references and replaced with +BATT references.
Parts:
- added C? (x2): 15pF, symbol Device:C_Small
- added C? (x2): 0.1uF, Capacitors_SMD:C_0603, symbol Device:C_Small
- added C? (x2): 1uF, Capacitors_SMD:C_0603, symbol Device:C_Small
- added J?: Conn CAN, symbol Connector_Generic:Conn_01x03
- added R? (x2): 10k, symbol Device:R_Small_US
- added U?: MCP2515, Package_SO:TSSOP-20_4.4x6.5mm_P0.65mm, symbol MCU_Powertrain:MCP2515-QFN20
- added U?: SN65HVD232, Package_SO:SOIC-8_3.9x4.9mm_P1.27mm, symbol Interface_CAN_LIN:SN65HVD232
- added Y?: 20MHz, symbol Device:Crystal_Small
Connections:
- wire segments 104 -> 168
- no-connect marks 1 -> 7
Other:
- note added: "CAN chips decoupling cap"
- moved on the sheet: C?, D?, J?, L?, R?

Commit message: TI_MCU Updates
- Connected GPIO12 to CAN_INT, made switch active low so that it can test the interrupt.
- Connected SPI CS_1 to GPIO32
Parts:
- added H? (x4): MountingHole, symbol Mechanical:MountingHole
- R?: value 68.0kΩ -> 68.0k
- R?: value 20.0kΩ -> 20.0k
- R?: value 330Ω -> 330
Connections:
- net labels added: CANH, CANL, RXCAN, TXCAN
Other:
- moved on the sheet: J?
Changed lines of the file:
@@
 AR Path="/5E56729B" Ref="R?"  Part="1"
 F 0 "R?" H 4350 5600 50  0000 L CNN
-F 1 "68.0kΩ" H 4350 5525 50  0000 L CNN
+F 1 "68.0k" H 4350 5525 50  0000 L CNN
 F 2 "Resistors_SMD:R_0603" V 4340 5590 50  0001 C CNN
 F 3 "~" H 4300 5600 50  0001 C CNN
@@
 AR Path="/5E5672C2" Ref="R?"  Part="1"
 F 0 "R?" H 5350 5450 50  0000 L CNN
-F 1 "330Ω" H 5350 5375 50  0000 L CNN
+F 1 "330" H 5350 5375 50  0000 L CNN
 F 2 "Resistors_SMD:R_0603" V 5340 5440 50  0001 C CNN
 F 3 "~" H 5300 5450 50  0001 C CNN
@@
 	6550 4125 7650 4125
 Wire Wire Line
-	8250 3575 8250 3500
+	8250 3575 8250 3550
 $Comp
 L power:+3V3 #PWR?
 U 1 1 5E4011A5
-P 8250 3500
+P 8250 3550
 AR Path="/5E20A2BB/5E4011A5" Ref="#PWR?"  Part="1"
 AR Path="/5E4011A5" Ref="#PWR?"  Part="1"
-F 0 "#PWR?" H 8250 3350 50  0001 C CNN
-F 1 "+3V3" H 8375 3575 50  0000 C CNN
-F 2 "" H 8250 3500 50  0001 C CNN
-F 3 "" H 8250 3500 50  0001 C CNN
-	1    8250 3500
+F 0 "#PWR?" H 8250 3400 50  0001 C CNN
+F 1 "+3V3" H 8225 3700 50  0000 C CNN
+F 2 "" H 8250 3550 50  0001 C CNN
+F 3 "" H 8250 3550 50  0001 C CNN
+	1    8250 3550
 	1    0    0    -1
 $EndComp
@@
 AR Path="/5E420A93" Ref="#PWR?"  Part="1"
 F 0 "#PWR?" H 9075 4425 50  0001 C CNN
-F 1 "+3V3" H 9200 4650 50  0000 C CNN
+F 1 "+3V3" H 9075 4725 50  0000 C CNN
 F 2 "" H 9075 4575 50  0001 C CNN
 F 3 "" H 9075 4575 50  0001 C CNN
@@
 AR Path="/5E5672A2" Ref="R?"  Part="1"
 F 0 "R?" H 4350 6000 50  0000 L CNN
-F 1 "20.0kΩ" H 4350 5925 50  0000 L CNN
+F 1 "20.0k" H 4350 5925 50  0000 L CNN
 F 2 "Resistors_SMD:R_0603" V 4340 5990 50  0001 C CNN
 F 3 "~" H 4300 6000 50  0001 C CNN
@@
 $EndComp
 $Comp
-L power:+3V3 #PWR?
-U 1 1 5E49D988
-P 9825 3575
-AR Path="/5E20A2BB/5E49D988" Ref="#PWR?"  Part="1"
-AR Path="/5E49D988" Ref="#PWR?"  Part="1"
-F 0 "#PWR?" H 9825 3425 50  0001 C CNN
-F 1 "+3V3" H 9950 3650 50  0000 C CNN
-F 2 "" H 9825 3575 50  0001 C CNN
-F 3 "" H 9825 3575 50  0001 C CNN
-	1    9825 3575
-	1    0    0    -1
-$EndComp
-Wire Wire Line
-	9825 3575 9825 3625
-$Comp
 L power:GND #PWR?
 U 1 1 5E4A3E7B
@@
 L Connector_Generic:Conn_01x03 J?
 U 1 1 5E4DDF4C
-P 10650 4025
-F 0 "J?" H 10730 4067 50  0000 L CNN
-F 1 "Conn CAN" H 10730 3976 50  0000 L CNN
-F 2 "" H 10650 4025 50  0001 C CNN
-F 3 "~" H 10650 4025 50  0001 C CNN
-	1    10650 4025
-	1    0    0    -1
-$EndComp
-Wire Wire Line
-	10225 3925 10450 3925
-Wire Wire Line
-	10225 4025 10450 4025
-Wire Wire Line
-	10450 4125 10375 4125
+P 10775 4025
+F 0 "J?" H 10855 4067 50  0000 L CNN
+F 1 "Conn CAN" H 10855 3976 50  0000 L CNN
+F 2 "" H 10775 4025 50  0001 C CNN
+F 3 "~" H 10775 4025 50  0001 C CNN
+	1    10775 4025
+	1    0    0    -1
+$EndComp
+Wire Wire Line
+	10225 3925 10575 3925
+Wire Wire Line
+	10225 4025 10575 4025
+Wire Wire Line
+	10575 4125 10375 4125
 Wire Wire Line
 	10375 4125 10375 4200
@@
 AR Path="/5E4FE87C" Ref="#PWR?"  Part="1"
 F 0 "#PWR?" H 6125 3775 50  0001 C CNN
-F 1 "+3V3" H 6250 4000 50  0000 C CNN
+F 1 "+3V3" H 6125 4075 50  0000 C CNN
 F 2 "" H 6125 3925 50  0001 C CNN
 F 3 "" H 6125 3925 50  0001 C CNN
@@
 	1    0    0    -1
 $EndComp
+$Comp
+L Mechanical:MountingHole H?
+U 1 1 5E668803
+P 1175 6750
+F 0 "H?" H 1275 6796 50  0000 L CNN
+F 1 "MountingHole" H 1275 6705 50  0000 L CNN
+F 2 "" H 1175 6750 50  0001 C CNN
+F 3 "~" H 1175 6750 50  0001 C CNN
+	1    1175 6750
+	1    0    0    -1
+$EndComp
+$Comp
+L Mechanical:MountingHole H?
+U 1 1 5E669612
+P 1950 6750
+F 0 "H?" H 2050 6796 50  0000 L CNN
+F 1 "MountingHole" H 2050 6705 50  0000 L CNN
+F 2 "" H 1950 6750 50  0001 C CNN
+F 3 "~" H 1950 6750 50  0001 C CNN
+	1    1950 6750
+	1    0    0    -1
+$EndComp
+$Comp
+L Mechanical:MountingHole H?
+U 1 1 5E669ABC
+P 2725 6750
+F 0 "H?" H 2825 6796 50  0000 L CNN
+F 1 "MountingHole" H 2825 6705 50  0000 L CNN
+F 2 "" H 2725 6750 50  0001 C CNN
+F 3 "~" H 2725 6750 50  0001 C CNN
+	1    2725 6750
+	1    0    0    -1
+$EndComp
+$Comp
+L Mechanical:MountingHole H?
+U 1 1 5E669F85
+P 3500 6750
+F 0 "H?" H 3600 6796 50  0000 L CNN
+F 1 "MountingHole" H 3600 6705 50  0000 L CNN
+F 2 "" H 3500 6750 50  0001 C CNN
+F 3 "~" H 3500 6750 50  0001 C CNN
+	1    3500 6750
+	1    0    0    -1
+$EndComp
+Text Label 10300 3925 0    50   ~ 0
+CANH
+Text Label 10300 4025 0    50   ~ 0
+CANL
+Text Label 9025 3825 0    50   ~ 0
+TXCAN
+Text Label 9025 3925 0    50   ~ 0
+RXCAN
+Wire Wire Line
+	9825 3600 9825 3625
+$Comp
+L power:+3V3 #PWR?
+U 1 1 5E49D988
+P 9825 3600
+AR Path="/5E20A2BB/5E49D988" Ref="#PWR?"  Part="1"
+AR Path="/5E49D988" Ref="#PWR?"  Part="1"
+F 0 "#PWR?" H 9825 3450 50  0001 C CNN
+F 1 "+3V3" H 9825 3750 50  0000 C CNN
+F 2 "" H 9825 3600 50  0001 C CNN
+F 3 "" H 9825 3600 50  0001 C CNN
+	1    9825 3600
+	1    0    0    -1
+$EndComp

Commit message: Testpoints
- Added Testpoints everywhere!
- Schematic is "done" and any mistakes should be able to be corrected with small bodges later
Parts:
- added TP? (x21): TestPoint, symbol Connector:TestPoint
Connections:
- wire segments 168 -> 216
Other:
- moved on the sheet: C?, D?, H?, J?, L?, R?

Commit message: Completed BOM
- Added Digikey PNs to each component.
- Removed double 3V3 LED indicator
Parts:
- removed C?: 1uF, Capacitors_SMD:C_0603, symbol Device:C_Small
- removed TP? (x9): TestPoint, symbol Connector:TestPoint
- added C29: 1uF, Capacitors_SMD:C_0805, symbol Device:C_Small
- added TP10, TP11, TP13, TP14, TP15, TP5, TP7, TP8, TP9: TestPoint, symbol Connector:TestPoint
- C21, C22: renamed from C?; footprint (none) -> Capacitors_SMD:C_0603; Digikey (none) -> 311-1060-1-ND
- C28: renamed from C?; footprint Capacitors_SMD:C_0603 -> Capacitors_SMD:C_0805; Digikey (none) -> 399-8011-1-ND
- J1: renamed from J?; footprint ESC Drivetrain V1:3mm_Bullet_A -> (none)
- J2: renamed from J?; footprint ESC Drivetrain V1:3mm_Bullet_B -> (none)
- J3: renamed from J?; footprint ESC Drivetrain V1:3mm_Bullet_C -> (none)
- J4: renamed from J?; Digikey (none) -> 302-S101
- J6: renamed from J?; Digikey (none) -> WM4901-ND
- R17, R18: renamed from R?; Digikey (none) -> 311-10.0KCRCT-ND
- R19: renamed from R?; Digikey (none) -> A129743CT-ND
- TP1, TP2, TP3: renamed from TP?; Digikey (none) -> 36-5117-ND
- TP12, TP6: renamed from TP?; Digikey (none) -> 36-5119-ND
- TP16, TP17, TP19, TP21, TP4: renamed from TP?; Digikey (none) -> 36-5001-ND
- TP18, TP20: renamed from TP?; Digikey (none) -> 36-5000-ND
- gave numbers to parts that had none: 20

Commit message: Assigned Footprints
- All footprints assigned
- Created RA 3mm bullet fooprint, may need to adjust it later
- Fixed errors
Parts:
- H1, H2, H3, H4: footprint (none) -> Mounting_Holes:MountingHole_3mm_Pad_Via
- J1, J2, J3: footprint (none) -> MCU_Powertrain:3mm_Bullet_RA
- J4: footprint (none) -> MCU_Powertrain:2x05_Prog_Header
- J5: footprint (none) -> Connectors:Tag-Connect_TC2050-IDC-NL
- J6: footprint (none) -> MCU_Powertrain:70553-03
- J7: footprint (none) -> MCU_Powertrain:AMASS_XT60-M
- L1: footprint ESC Drivetrain V1:Eaton_Inductor -> MCU_Powertrain:Eaton_Inductor
- R17, R18: footprint (none) -> Resistors_SMD:R_0805
- TP1, TP10, TP11, TP12, TP13, TP14, TP15, TP16, TP17, TP18, TP19, TP2, TP20, TP21, TP3, TP4, TP5, TP6, TP7, TP8, TP9: footprint (none) -> Testpoints:TestPoint_Loop_D1.80mm_Drill1.0mm_Beaded
- U2: footprint Package_SO:SOIC-8_3.9x4.9mm_P1.27mm -> Housings_SOIC:SOIC-8_3.9x4.9mm_Pitch1.27mm
- U3: footprint Package_SO:TSSOP-20_4.4x6.5mm_P0.65mm -> Housings_DFN_QFN:QFN-20-1EP_4x4mm_Pitch0.5mm
- Y1: footprint (none) -> Crystals:Crystal_SMD_SeikoEpson_TSX3225-4pin_3.2x2.5mm
