File: PCBs/MCU_Powertrain/Powertrain.sch (KiCad schematic (older format))
At the start: 68 parts, among them J1 PHASE_A, J2 Conn_01x02, J3 PHASE_B, J4 PHASE_C, J5 Conn_02x10_Odd_Even, J6 Conn_02x10_Odd_Even, J7 I2C Header, Q1 SIZF906DT, Q2 SIZF906DT, Q3 SIZF906DT, U1 DRV8305, U2 LMR16006XDDC

Commit message: More Schematic Changes
- Connected TI_MCU schematic to Powertrain schematic
- Added power input
Parts:
- removed C21: 22uF, Capacitors_SMD:C_0805, symbol Device:C_Small
- removed C22: 0.33uF, Capacitors_SMD:C_0603, symbol Device:C_Small
- removed C23: 0.1uF, Capacitors_SMD:C_0603, symbol Device:C_Small
- removed D3: GREEN, LEDs:LED_0603, symbol Device:LED_ALT
- removed D4: D_Schottky_ALT, Diodes_SMD:D_SOD-123F, symbol Device:D_Schottky_ALT
- removed J1: PHASE_A, ESC Drivetrain V1:3mm_Bullet_A, symbol Connector_Generic:Conn_01x01
- removed J2: Conn_01x02, ESC Drivetrain V1:AMASS_XT60-M, symbol Connector_Generic:Conn_01x02
- removed J3: PHASE_B, ESC Drivetrain V1:3mm_Bullet_B, symbol Connector_Generic:Conn_01x01
- removed J4: PHASE_C, ESC Drivetrain V1:3mm_Bullet_C, symbol Connector_Generic:Conn_01x01
- removed J5, J6: Conn_02x10_Odd_Even, ESC Drivetrain V1:Pin_Header_Straight_2x10_Pitch2.54mm_LaunchPad, symbol Connector_Generic:Conn_02x10_Odd_Even
- removed J7: I2C Header, Pin_Headers:Pin_Header_Straight_1x03_Pitch2.54mm, symbol Connector_Generic:Conn_01x03
- removed L1: 15uH, ESC Drivetrain V1:Eaton_Inductor, symbol Device:L_Core_Ferrite
- removed R17: 330Ω, Resistors_SMD:R_0603, symbol Device:R_US
- removed R18: 68.0kΩ, Resistors_SMD:R_0603, symbol Device:R_US
- removed R19: 20.0kΩ, Resistors_SMD:R_0603, symbol Device:R_US
- removed R23, R24: 2.7kΩ, Resistors_SMD:R_0603, symbol Device:R_US
- removed U2: LMR16006XDDC, TO_SOT_Packages_SMD:SOT-23-6, symbol ESC~Drivetrain~V1:LMR16006XDDC
Connections:
- net labels added: +BATT, Phase_A, Phase_B, Phase_C, SPI_CLK, SPI_CS, SPI_MISO, SPI_MOSI
- net labels removed: ADC_IN, SCL_EXTERN, SDA_EXTERN
- wire segments 314 -> 250
- no-connect marks 14 -> 0
Other:
- note added: "External Signals"
- note added: "Test different cap values, try to minimize cap size and cost!"
- note removed: "3.3V Regulator"
- note removed: "Headers and Protection"
- note removed: "Optional Pullup Resistors"
- note removed: "SCL = SCLA, GPIO 33"
- note removed: "SDA = SDAA, GPIO 32"
- moved on the sheet: C24, C25, C26, R20, R21, R22

Commit message: CAN and Minor Changes
- Added CAN Controller (MCP2515) and CAN transciever
- Added net-ties to shunts
- Removed all +12V references and replaced with +BATT references.
Parts:
- added NT? (x3): Net-Tie_2, symbol Device:Net-Tie_2
Connections:
- net labels added: SPI_CS_0
- net labels removed: +12V, SPI_CS
- wire segments 250 -> 253
Changed lines of the file:
@@
 Connection ~ 1700 800
-$Comp
-L power:+12V #PWR01
-U 1 1 5D54F21B
-P 1700 750
-F 0 "#PWR01" H 1700 600 50  0001 C CNN
-F 1 "+12V" H 1715 923 50  0000 C CNN
-F 2 "" H 1700 750 50  0001 C CNN
-F 3 "" H 1700 750 50  0001 C CNN
-	1    1700 750
-	1    0    0    -1
-$EndComp
 $Comp
 L power:GND #PWR08
@@
 	1    0    0    -1
 $EndComp
-$Comp
-L power:+12V #PWR025
-U 1 1 5D571885
-P 1400 4200
-F 0 "#PWR025" H 1400 4050 50  0001 C CNN
-F 1 "+12V" H 1415 4373 50  0000 C CNN
-F 2 "" H 1400 4200 50  0001 C CNN
-F 3 "" H 1400 4200 50  0001 C CNN
-	1    1400 4200
-	1    0    0    -1
-$EndComp
 Wire Wire Line
 	1400 4200 1400 4225
@@
 Wire Wire Line
 	4025 1925 4025 1850
-$Comp
-L power:+12V #PWR012
-U 1 1 5D5A2AFD
-P 4025 1850
-F 0 "#PWR012" H 4025 1700 50  0001 C CNN
-F 1 "+12V" H 4025 2000 50  0000 C CNN
-F 2 "" H 4025 1850 50  0001 C CNN
-F 3 "" H 4025 1850 50  0001 C CNN
-	1    4025 1850
-	1    0    0    -1
-$EndComp
 Wire Wire Line
 	3200 1825 3875 1825
@@
 Wire Wire Line
 	6100 2225 6100 2075
-Wire Wire Line
-	6100 2575 6100 2650
-Wire Wire Line
-	6100 2650 5550 2650
-Wire Wire Line
-	6100 2650 6100 2800
-Connection ~ 6100 2650
 Text Label 5550 2225 0    50   ~ 0
 SN1
-Text Label 5550 2650 0    50   ~ 0
-SP1
 $Comp
 L power:GND #PWR020
@@
 Wire Wire Line
 	8050 2200 8050 2050
-Wire Wire Line
-	8050 2550 8050 2625
-Wire Wire Line
-	8050 2625 7500 2625
-Wire Wire Line
-	8050 2625 8050 2775
-Connection ~ 8050 2625
 $Comp
 L power:GND #PWR014
@@
 	9975 2550 9975 2625
 Wire Wire Line
-	9975 2625 9425 2625
+	9975 2625 9825 2625
 Wire Wire Line
 	9975 2625 9975 2775
@@
 Connection ~ 7550 3625
 $Comp
-L power:+12V #PWR09
-U 1 1 5E0EF3BA
-P 5100 1625
-F 0 "#PWR09" H 5100 1475 50  0001 C CNN
-F 1 "+12V" H 5115 1798 50  0000 C CNN
-F 2 "" H 5100 1625 50  0001 C CNN
-F 3 "" H 5100 1625 50  0001 C CNN
-	1    5100 1625
-	1    0    0    -1
-$EndComp
-$Comp
 L Device:LED_ALT D1
 U 1 1 5E0F0E06
@@
 	4675 4700 4675 500
 Wire Notes Line
-	6925 7750 525  7750
+	4625 7750 525  7750
 Wire Notes Line
 	500  7750 500  5325
@@
 	1000 7425 1300 7425
 Text HLabel 3475 6025 0    50   Input ~ 0
-SPI_CS
+SPI_CS_0
 Text HLabel 3475 6125 0    50   BiDi ~ 0
 SPI_MOSI
@@
 Text HLabel 3475 6850 0    50   Output ~ 0
 nFAULT
+Wire Notes Line
+	500  5325 4625 5325
+Wire Notes Line
+	4625 5325 4625 7750
+$Comp
+L power:+BATT #PWR?
+U 1 1 5E32BA5B
+P 1700 750
+F 0 "#PWR?" H 1700 600 50  0001 C CNN
+F 1 "+BATT" H 1715 923 50  0000 C CNN
+F 2 "" H 1700 750 50  0001 C CNN
+F 3 "" H 1700 750 50  0001 C CNN
+	1    1700 750
+	1    0    0    -1
+$EndComp
+$Comp
+L power:+BATT #PWR?
+U 1 1 5E32C321
+P 4025 1850
+F 0 "#PWR?" H 4025 1700 50  0001 C CNN
+F 1 "+BATT" H 4040 2023 50  0000 C CNN
+F 2 "" H 4025 1850 50  0001 C CNN
+F 3 "" H 4025 1850 50  0001 C CNN
+	1    4025 1850
+	1    0    0    -1
+$EndComp
+$Comp
+L power:+BATT #PWR?
+U 1 1 5E32CCC5
+P 5100 1625
+F 0 "#PWR?" H 5100 1475 50  0001 C CNN
+F 1 "+BATT" H 5115 1798 50  0000 C CNN
+F 2 "" H 5100 1625 50  0001 C CNN
+F 3 "" H 5100 1625 50  0001 C CNN
+	1    5100 1625
+	1    0    0    -1
+$EndComp
+$Comp
+L power:+BATT #PWR?
+U 1 1 5E32DA12
+P 1400 4200
+F 0 "#PWR?" H 1400 4050 50  0001 C CNN
+F 1 "+BATT" H 1415 4373 50  0000 C CNN
+F 2 "" H 1400 4200 50  0001 C CNN
+F 3 "" H 1400 4200 50  0001 C CNN
+	1    1400 4200
+	1    0    0    -1
+$EndComp
+$Comp
+L Device:Net-Tie_2 NT?
+U 1 1 5E373C00
+P 5825 2650
+F 0 "NT?" H 5825 2700 50  0000 C CNN
+F 1 "Net-Tie_2" H 5825 2550 50  0001 C CNN
+F 2 "" H 5825 2650 50  0001 C CNN
+F 3 "~" H 5825 2650 50  0001 C CNN
+	1    5825 2650
+	1    0    0    -1
+$EndComp
+Text Label 5550 2650 0    50   ~ 0
+SP1
+Wire Wire Line
+	6100 2575 6100 2650
+Wire Wire Line
+	5550 2650 5725 2650
+Wire Wire Line
+	5925 2650 6100 2650
+Connection ~ 6100 2650
+Wire Wire Line
+	6100 2650 6100 2800
+$Comp
+L Device:Net-Tie_2 NT?
+U 1 1 5E39434A
+P 7775 2625
+F 0 "NT?" H 7775 2675 50  0000 C CNN
+F 1 "Net-Tie_2" H 7775 2525 50  0001 C CNN
+F 2 "" H 7775 2625 50  0001 C CNN
+F 3 "~" H 7775 2625 50  0001 C CNN
+	1    7775 2625
+	1    0    0    -1
+$EndComp
+Wire Wire Line
+	8050 2550 8050 2625
+Wire Wire Line
+	7500 2625 7675 2625
+Wire Wire Line
+	7875 2625 8050 2625
+Connection ~ 8050 2625
+Wire Wire Line
+	8050 2625 8050 2775
+Wire Wire Line
+	9625 2625 9425 2625
+$Comp
+L Device:Net-Tie_2 NT?
+U 1 1 5E3B408A
+P 9725 2625
+F 0 "NT?" H 9725 2675 50  0000 C CNN
+F 1 "Net-Tie_2" H 9725 2525 50  0001 C CNN
+F 2 "" H 9725 2625 50  0001 C CNN
+F 3 "~" H 9725 2625 50  0001 C CNN
+	1    9725 2625
+	1    0    0    -1
+$EndComp
 $EndSCHEMATC

Commit message: TI_MCU Updates
- Connected GPIO12 to CAN_INT, made switch active low so that it can test the interrupt.
- Connected SPI CS_1 to GPIO32
Parts:
- R1, R6: value 10kΩ -> 10k
- R10: value 330Ω -> 330
- R11, R8, R9: value 5mΩ -> 5m
- R12, R13, R14, R16: value 4.99kΩ -> 4.99k
- R15, R3, R4, R5: value 22.0kΩ -> 22.0k
- R2: value 100Ω -> 100
- R20, R21, R22: value 56Ω -> 56
- R7: value 2.7kΩ -> 2.7k
Changed lines of the file:
@@
 P 950 2425
 F 0 "R10" H 1018 2471 50  0000 L CNN
-F 1 "330Ω" H 1018 2380 50  0000 L CNN
+F 1 "330" H 1018 2380 50  0000 L CNN
 F 2 "Resistors_SMD:R_0603" V 990 2415 50  0001 C CNN
 F 3 "~" H 950 2425 50  0001 C CNN
@@
 U 1 1 5D55E30C
 P 750 2200
-F 0 "R6" H 525 2250 50  0000 L CNN
-F 1 "10kΩ" H 500 2150 50  0000 L CNN
+F 0 "R6" H 550 2250 50  0000 L CNN
+F 1 "10k" H 525 2150 50  0000 L CNN
 F 2 "Resistors_SMD:R_0603" V 790 2190 50  0001 C CNN
 F 3 "~" H 750 2200 50  0001 C CNN
@@
 P 3700 1925
 F 0 "R2" V 3775 1825 50  0000 C CNN
-F 1 "100Ω" V 3775 2050 50  0000 C CNN
+F 1 "100" V 3775 2050 50  0000 C CNN
 F 2 "Resistors_SMD:R_0603" V 3740 1915 50  0001 C CNN
 F 3 "~" H 3700 1925 50  0001 C CNN
@@
 P 3875 1525
 F 0 "R1" H 3925 1575 50  0000 L CNN
-F 1 "10kΩ" H 3925 1500 50  0000 L CNN
+F 1 "10k" H 3925 1500 50  0000 L CNN
 F 2 "Resistors_SMD:R_0603" V 3915 1515 50  0001 C CNN
 F 3 "~" H 3875 1525 50  0001 C CNN
@@
 P 2125 5975
 F 0 "R20" V 2075 5800 50  0000 C CNN
-F 1 "56Ω" V 2075 6150 50  0000 C CNN
+F 1 "56" V 2075 6150 50  0000 C CNN
 F 2 "Resistors_SMD:R_0603" V 2165 5965 50  0001 C CNN
 F 3 "~" H 2125 5975 50  0001 C CNN
@@
 P 7925 4225
 F 0 "R16" H 7975 4225 50  0000 L CNN
-F 1 "4.99kΩ" H 7975 4150 50  0000 L CNN
+F 1 "4.99k" H 7975 4150 50  0000 L CNN
 F 2 "Resistors_SMD:R_0603" V 7965 4215 50  0001 C CNN
 F 3 "~" H 7925 4225 50  0001 C CNN
@@
 P 6100 2425
 F 0 "R11" H 6168 2471 50  0000 L CNN
-F 1 "5mΩ" H 6168 2380 50  0000 L CNN
+F 1 "5m" H 6168 2380 50  0000 L CNN
 F 2 "ESC Drivetrain V1:R_2512_Sense" V 6140 2415 50  0001 C CNN
 F 3 "" H 6100 2425 50  0001 C CNN
@@
 P 6475 2125
 F 0 "R5" H 6543 2171 50  0000 L CNN
-F 1 "22.0kΩ" H 6543 2080 50  0000 L CNN
+F 1 "22.0k" H 6543 2080 50  0000 L CNN
 F 2 "Resistors_SMD:R_0603" V 6515 2115 50  0001 C CNN
 F 3 "~" H 6475 2125 50  0001 C CNN
@@
 P 6475 2525
 F 0 "R14" H 6525 2525 50  0000 L CNN
-F 1 "4.99kΩ" H 6525 2450 50  0000 L CNN
+F 1 "4.99k" H 6525 2450 50  0000 L CNN
 F 2 "Resistors_SMD:R_0603" V 6515 2515 50  0001 C CNN
 F 3 "~" H 6475 2525 50  0001 C CNN
@@
 P 8050 2400
 F 0 "R8" H 8118 2446 50  0000 L CNN
-F 1 "5mΩ" H 8118 2355 50  0000 L CNN
+F 1 "5m" H 8118 2355 50  0000 L CNN
 F 2 "ESC Drivetrain V1:R_2512_Sense" V 8090 2390 50  0001 C CNN
 F 3 "" H 8050 2400 50  0001 C CNN
@@
 P 8425 2500
 F 0 "R12" H 8475 2500 50  0000 L CNN
-F 1 "4.99kΩ" H 8475 2425 50  0000 L CNN
+F 1 "4.99k" H 8475 2425 50  0000 L CNN
 F 2 "Resistors_SMD:R_0603" V 8465 2490 50  0001 C CNN
 F 3 "~" H 8425 2500 50  0001 C CNN
@@
 P 9975 2400
 F 0 "R9" H 10043 2446 50  0000 L CNN
-F 1 "5mΩ" H 10043 2355 50  0000 L CNN
+F 1 "5m" H 10043 2355 50  0000 L CNN
 F 2 "ESC Drivetrain V1:R_2512_Sense" V 10015 2390 50  0001 C CNN
 F 3 "" H 9975 2400 50  0001 C CNN
@@
 P 10350 2500
 F 0 "R13" H 10400 2500 50  0000 L CNN
-F 1 "4.99kΩ" H 10400 2425 50  0000 L CNN
+F 1 "4.99k" H 10400 2425 50  0000 L CNN
 F 2 "Resistors_SMD:R_0603" V 10390 2490 50  0001 C CNN
 F 3 "~" H 10350 2500 50  0001 C CNN
@@
 P 5100 2225
 F 0 "R7" H 5150 2225 50  0000 L CNN
-F 1 "2.7kΩ" H 5150 2150 50  0000 L CNN
+F 1 "2.7k" H 5150 2150 50  0000 L CNN
 F 2 "Resistors_SMD:R_0603" V 5140 2215 50  0001 C CNN
 F 3 "~" H 5100 2225 50  0001 C CNN
@@
 Wire Notes Line
 	500  7750 500  5325
-Wire Notes Line
-	11125 4750 11125 6500
 Text Notes 4725 675  0    79   Italic 16
 H-Bridges and VIN
@@
 P 2125 6075
 F 0 "R21" V 2075 5900 50  0000 C CNN
-F 1 "56Ω" V 2075 6250 50  0000 C CNN
+F 1 "56" V 2075 6250 50  0000 C CNN
 F 2 "Resistors_SMD:R_0603" V 2165 6065 50  0001 C CNN
 F 3 "~" H 2125 6075 50  0001 C CNN
@@
 P 2125 6175
 F 0 "R22" V 2075 6000 50  0000 C CNN
-F 1 "56Ω" V 2075 6350 50  0000 C CNN
+F 1 "56" V 2075 6350 50  0000 C CNN
 F 2 "Resistors_SMD:R_0603" V 2165 6165 50  0001 C CNN
 F 3 "~" H 2125 6175 50  0001 C CNN
@@
 P 8425 2100
 F 0 "R3" H 8493 2146 50  0000 L CNN
-F 1 "22.0kΩ" H 8493 2055 50  0000 L CNN
+F 1 "22.0k" H 8493 2055 50  0000 L CNN
 F 2 "Resistors_SMD:R_0603" V 8465 2090 50  0001 C CNN
 F 3 "~" H 8425 2100 50  0001 C CNN
@@
 P 10350 2100
 F 0 "R4" H 10418 2146 50  0000 L CNN
-F 1 "22.0kΩ" H 10418 2055 50  0000 L CNN
+F 1 "22.0k" H 10418 2055 50  0000 L CNN
 F 2 "Resistors_SMD:R_0603" V 10390 2090 50  0001 C CNN
 F 3 "~" H 10350 2100 50  0001 C CNN
@@
 P 7925 3825
 F 0 "R15" H 7993 3871 50  0000 L CNN
-F 1 "22.0kΩ" H 7993 3780 50  0000 L CNN
+F 1 "22.0k" H 7993 3780 50  0000 L CNN
 F 2 "Resistors_SMD:R_0603" V 7965 3815 50  0001 C CNN
 F 3 "~" H 7925 3825 50  0001 C CNN
@@
 P 4425 1550
 F 0 "C27" H 4255 1640 50  0000 L CNN
-F 1 "1uF" H 4215 1560 50  0000 L CNN
+F 1 "1uF" H 4250 1475 50  0000 L CNN
 F 2 "Capacitors_SMD:C_0603" H 4425 1550 50  0001 C CNN
 F 3 "" H 4425 1550 50  0001 C CNN

Commit message: Completed BOM
- Added Digikey PNs to each component.
- Removed double 3V3 LED indicator
Parts:
- gave numbers to parts that had none: 3
Changed lines of the file:
@@
 $EndComp
 $Comp
-L power:+BATT #PWR?
+L power:+BATT #PWR0134
 U 1 1 5E588C2B
 P 5900 3525
-F 0 "#PWR?" H 5900 3375 50  0001 C CNN
+F 0 "#PWR0134" H 5900 3375 50  0001 C CNN
 F 1 "+BATT" H 5915 3698 50  0000 C CNN
 F 2 "" H 5900 3525 50  0001 C CNN
@@
 Test different cap values, try to minimize cap size and cost!
 $Comp
-L power:+BATT #PWR?
+L power:+BATT #PWR0135
 U 1 1 5E58A9D0
 P 6100 1000
-F 0 "#PWR?" H 6100 850 50  0001 C CNN
+F 0 "#PWR0135" H 6100 850 50  0001 C CNN
 F 1 "+BATT" H 6115 1173 50  0000 C CNN
 F 2 "" H 6100 1000 50  0001 C CNN
@@
 $EndComp
 $Comp
-L power:+BATT #PWR?
+L power:+BATT #PWR0136
 U 1 1 5E58B583
 P 8050 975
-F 0 "#PWR?" H 8050 825 50  0001 C CNN
+F 0 "#PWR0136" H 8050 825 50  0001 C CNN
 F 1 "+BATT" H 8065 1148 50  0000 C CNN
 F 2 "" H 8050 975 50  0001 C CNN
@@
 $EndComp
 $Comp
-L power:+BATT #PWR?
+L power:+BATT #PWR0137
 U 1 1 5E58BD6D
 P 9975 975
-F 0 "#PWR?" H 9975 825 50  0001 C CNN
+F 0 "#PWR0137" H 9975 825 50  0001 C CNN
 F 1 "+BATT" H 9990 1148 50  0000 C CNN
 F 2 "" H 9975 975 50  0001 C CNN
@@
 	4625 5325 4625 7750
 $Comp
-L power:+BATT #PWR?
+L power:+BATT #PWR0138
 U 1 1 5E32BA5B
 P 1700 750
-F 0 "#PWR?" H 1700 600 50  0001 C CNN
+F 0 "#PWR0138" H 1700 600 50  0001 C CNN
 F 1 "+BATT" H 1715 923 50  0000 C CNN
 F 2 "" H 1700 750 50  0001 C CNN
@@
 $EndComp
 $Comp
-L power:+BATT #PWR?
+L power:+BATT #PWR0139
 U 1 1 5E32C321
 P 4025 1850
-F 0 "#PWR?" H 4025 1700 50  0001 C CNN
+F 0 "#PWR0139" H 4025 1700 50  0001 C CNN
 F 1 "+BATT" H 4040 2023 50  0000 C CNN
 F 2 "" H 4025 1850 50  0001 C CNN
@@
 $EndComp
 $Comp
-L power:+BATT #PWR?
+L power:+BATT #PWR0140
 U 1 1 5E32CCC5
 P 5100 1625
-F 0 "#PWR?" H 5100 1475 50  0001 C CNN
+F 0 "#PWR0140" H 5100 1475 50  0001 C CNN
 F 1 "+BATT" H 5115 1798 50  0000 C CNN
 F 2 "" H 5100 1625 50  0001 C CNN
@@
 $EndComp
 $Comp
-L power:+BATT #PWR?
+L power:+BATT #PWR0141
 U 1 1 5E32DA12
 P 1400 4200
-F 0 "#PWR?" H 1400 4050 50  0001 C CNN
+F 0 "#PWR0141" H 1400 4050 50  0001 C CNN
 F 1 "+BATT" H 1415 4373 50  0000 C CNN
 F 2 "" H 1400 4200 50  0001 C CNN
@@
 $EndComp
 $Comp
-L Device:Net-Tie_2 NT?
+L Device:Net-Tie_2 NT3
 U 1 1 5E373C00
 P 5825 2650
-F 0 "NT?" H 5825 2700 50  0000 C CNN
+F 0 "NT3" H 5825 2700 50  0000 C CNN
 F 1 "Net-Tie_2" H 5825 2550 50  0001 C CNN
 F 2 "" H 5825 2650 50  0001 C CNN
@@
 	6100 2650 6100 2800
 $Comp
-L Device:Net-Tie_2 NT?
+L Device:Net-Tie_2 NT1
 U 1 1 5E39434A
 P 7775 2625
-F 0 "NT?" H 7775 2675 50  0000 C CNN
+F 0 "NT1" H 7775 2675 50  0000 C CNN
 F 1 "Net-Tie_2" H 7775 2525 50  0001 C CNN
 F 2 "" H 7775 2625 50  0001 C CNN
@@
 	9625 2625 9425 2625
 $Comp
-L Device:Net-Tie_2 NT?
+L Device:Net-Tie_2 NT2
 U 1 1 5E3B408A
 P 9725 2625
-F 0 "NT?" H 9725 2675 50  0000 C CNN
+F 0 "NT2" H 9725 2675 50  0000 C CNN
 F 1 "Net-Tie_2" H 9725 2525 50  0001 C CNN
 F 2 "" H 9725 2625 50  0001 C CNN

Commit message: Assigned Footprints
- All footprints assigned
- Created RA 3mm bullet fooprint, may need to adjust it later
- Fixed errors
Parts:
- NT1, NT2, NT3: footprint (none) -> NetTies:NetTie-2_SMD_Pad0.5mm
- Q1, Q2, Q3: footprint ESC Drivetrain V1:SIZF906DT -> MCU_Powertrain:SIZF906DT
- R11, R8, R9: footprint ESC Drivetrain V1:R_2512_Sense -> MCU_Powertrain:R_2512_Sense
- U1: footprint ESC Drivetrain V1:DRV8305 -> MCU_Powertrain:DRV8305
Changed lines of the file:
@@
 F 0 "U1" H 2575 5706 79  0000 C CNN
 F 1 "DRV8305" H 2575 5571 79  0000 C CNN
-F 2 "ESC Drivetrain V1:DRV8305" H 2500 3825 79  0001 C CNN
+F 2 "MCU_Powertrain:DRV8305" H 2500 3825 79  0001 C CNN
 F 3 "http://www.ti.com/lit/ds/symlink/drv8305.pdf" H 4950 5425 79  0001 C CNN
 F 4 "296-42659-1-ND" H 4100 5275 79  0001 C CNN "Digikey"
@@
 F 0 "Q3" H 6225 1600 50  0000 L CNN
 F 1 "SIZF906DT" H 6225 1525 50  0000 L CNN
-F 2 "ESC Drivetrain V1:SIZF906DT" H 6200 1575 50  0001 C CNN
+F 2 "MCU_Powertrain:SIZF906DT" H 6200 1575 50  0001 C CNN
 F 3 "http://www.vishay.com/docs/67547/sizf906dt.pdf" H 6000 1475 50  0001 C CNN
 F 4 "SIZF906DT-T1-GE3CT-ND" H 6000 1425 50  0001 C CNN "Digikey"
@@
 F 0 "R11" H 6168 2471 50  0000 L CNN
 F 1 "5m" H 6168 2380 50  0000 L CNN
-F 2 "ESC Drivetrain V1:R_2512_Sense" V 6140 2415 50  0001 C CNN
+F 2 "MCU_Powertrain:R_2512_Sense" V 6140 2415 50  0001 C CNN
 F 3 "" H 6100 2425 50  0001 C CNN
 F 4 "YAG6124CT-ND" H 6100 2425 50  0001 C CNN "Digikey"
@@
 F 0 "Q1" H 8175 1575 50  0000 L CNN
 F 1 "SIZF906DT" H 8175 1500 50  0000 L CNN
-F 2 "ESC Drivetrain V1:SIZF906DT" H 8150 1550 50  0001 C CNN
+F 2 "MCU_Powertrain:SIZF906DT" H 8150 1550 50  0001 C CNN
 F 3 "http://www.vishay.com/docs/67547/sizf906dt.pdf" H 7950 1450 50  0001 C CNN
 F 4 "SIZF906DT-T1-GE3CT-ND" H 7950 1400 50  0001 C CNN "Digikey"
@@
 F 0 "R8" H 8118 2446 50  0000 L CNN
 F 1 "5m" H 8118 2355 50  0000 L CNN
-F 2 "ESC Drivetrain V1:R_2512_Sense" V 8090 2390 50  0001 C CNN
+F 2 "MCU_Powertrain:R_2512_Sense" V 8090 2390 50  0001 C CNN
 F 3 "" H 8050 2400 50  0001 C CNN
 F 4 "YAG6124CT-ND" H 8050 2400 50  0001 C CNN "Digikey"
@@
 F 0 "Q2" H 10100 1575 50  0000 L CNN
 F 1 "SIZF906DT" H 10100 1500 50  0000 L CNN
-F 2 "ESC Drivetrain V1:SIZF906DT" H 10075 1550 50  0001 C CNN
+F 2 "MCU_Powertrain:SIZF906DT" H 10075 1550 50  0001 C CNN
 F 3 "http://www.vishay.com/docs/67547/sizf906dt.pdf" H 9875 1450 50  0001 C CNN
 F 4 "SIZF906DT-T1-GE3CT-ND" H 9875 1400 50  0001 C CNN "Digikey"
@@
 F 0 "R9" H 10043 2446 50  0000 L CNN
 F 1 "5m" H 10043 2355 50  0000 L CNN
-F 2 "ESC Drivetrain V1:R_2512_Sense" V 10015 2390 50  0001 C CNN
+F 2 "MCU_Powertrain:R_2512_Sense" V 10015 2390 50  0001 C CNN
 F 3 "" H 9975 2400 50  0001 C CNN
 F 4 "YAG6124CT-ND" H 9975 2400 50  0001 C CNN "Digikey"
@@
 F 0 "NT3" H 5825 2700 50  0000 C CNN
 F 1 "Net-Tie_2" H 5825 2550 50  0001 C CNN
-F 2 "" H 5825 2650 50  0001 C CNN
+F 2 "NetTies:NetTie-2_SMD_Pad0.5mm" H 5825 2650 50  0001 C CNN
 F 3 "~" H 5825 2650 50  0001 C CNN
 	1    5825 2650
@@
 F 0 "NT1" H 7775 2675 50  0000 C CNN
 F 1 "Net-Tie_2" H 7775 2525 50  0001 C CNN
-F 2 "" H 7775 2625 50  0001 C CNN
+F 2 "NetTies:NetTie-2_SMD_Pad0.5mm" H 7775 2625 50  0001 C CNN
 F 3 "~" H 7775 2625 50  0001 C CNN
 	1    7775 2625
@@
 F 0 "NT2" H 9725 2675 50  0000 C CNN
 F 1 "Net-Tie_2" H 9725 2525 50  0001 C CNN
-F 2 "" H 9725 2625 50  0001 C CNN
+F 2 "NetTies:NetTie-2_SMD_Pad0.5mm" H 9725 2625 50  0001 C CNN
 F 3 "~" H 9725 2625 50  0001 C CNN
 	1    9725 2625
