File: PCBs/MCU_Powertrain/Powertrain.sch (KiCad schematic (older format))
At the start: 52 parts, among them Q1 SIZF906DT, Q2 SIZF906DT, Q3 SIZF906DT, U1 DRV8305

Commit message: Initial Layout, 3D Models, 0402s
- Changed C2, C4, C9, C16, C18 to 0402
- Some intial layout
- All 3D models added
Parts:
- added NT4, NT5, NT6: Net-Tie_2, MCU_Powertrain:NetTie-2_SMD_5mil, symbol Device:Net-Tie_2
- C16, C18, C9: footprint Capacitors_SMD:C_0603 -> Capacitors_SMD:C_0402; Digikey 1276-1018-1-ND -> 311-1036-1-ND
- C2, C4: footprint Capacitors_SMD:C_0603 -> Capacitors_SMD:C_0402; Digikey 399-7933-1-ND -> 490-10702-1-ND
- NT1, NT2, NT3: footprint NetTies:NetTie-2_SMD_Pad0.5mm -> MCU_Powertrain:NetTie-2_SMD_5mil
Connections:
- wire segments 253 -> 256
Changed lines of the file:
@@
 F 0 "C9" H 3675 3700 50  0000 L CNN
 F 1 "1000pF" H 3500 3625 50  0000 L CNN
-F 2 "Capacitors_SMD:C_0603" H 3850 3650 50  0001 C CNN
+F 2 "Capacitors_SMD:C_0402" H 3850 3650 50  0001 C CNN
 F 3 "" H 3850 3650 50  0001 C CNN
-F 4 "1276-1018-1-ND" H 3850 3650 50  0001 C CNN "Digikey"
+F 4 "311-1036-1-ND" H 3850 3650 50  0001 C CNN "Digikey"
 	1    3850 3650
 	1    0    0    -1
@@
 F 0 "C2" H 3225 1125 50  0000 L CNN
 F 1 "0.047uF" H 3025 1050 50  0000 L CNN
-F 2 "Capacitors_SMD:C_0603" H 3425 1050 50  0001 C CNN
+F 2 "Capacitors_SMD:C_0402" H 3425 1050 50  0001 C CNN
 F 3 "" H 3425 1050 50  0001 C CNN
-F 4 "399-7933-1-ND" H 3425 1050 50  0001 C CNN "Digikey"
+F 4 "490-10702-1-ND" H 3425 1050 50  0001 C CNN "Digikey"
 	1    3425 1050
 	-1   0    0    1
@@
 F 0 "C4" H 3225 1425 50  0000 L CNN
 F 1 "0.047uF" H 3025 1350 50  0000 L CNN
-F 2 "Capacitors_SMD:C_0603" H 3425 1350 50  0001 C CNN
+F 2 "Capacitors_SMD:C_0402" H 3425 1350 50  0001 C CNN
 F 3 "" H 3425 1350 50  0001 C CNN
-F 4 "399-7933-1-ND" H 3425 1350 50  0001 C CNN "Digikey"
+F 4 "490-10702-1-ND" H 3425 1350 50  0001 C CNN "Digikey"
 	1    3425 1350
 	-1   0    0    1
@@
 Text Label 5550 2075 0    50   ~ 0
 SL_A
-Wire Wire Line
-	6100 2275 6100 2225
 Connection ~ 6100 2075
-Wire Wire Line
-	5550 2225 6100 2225
-Connection ~ 6100 2225
-Wire Wire Line
-	6100 2225 6100 2075
 Text Label 5550 2225 0    50   ~ 0
 SN1
@@
 Wire Wire Line
 	8050 2050 7500 2050
-Wire Wire Line
-	8050 2250 8050 2200
 Connection ~ 8050 2050
-Wire Wire Line
-	7500 2200 8050 2200
-Connection ~ 8050 2200
-Wire Wire Line
-	8050 2200 8050 2050
 $Comp
 L power:GND #PWR014
@@
 Wire Wire Line
 	9975 2050 9425 2050
-Wire Wire Line
-	9975 2250 9975 2200
 Connection ~ 9975 2050
-Wire Wire Line
-	9425 2200 9975 2200
-Connection ~ 9975 2200
-Wire Wire Line
-	9975 2200 9975 2050
 Wire Wire Line
 	9975 2550 9975 2625
@@
 F 0 "C16" H 3625 4000 50  0000 L CNN
 F 1 "1000pF" H 3500 3925 50  0000 L CNN
-F 2 "Capacitors_SMD:C_0603" H 3850 3950 50  0001 C CNN
+F 2 "Capacitors_SMD:C_0402" H 3850 3950 50  0001 C CNN
 F 3 "" H 3850 3950 50  0001 C CNN
-F 4 "1276-1018-1-ND" H 3850 3950 50  0001 C CNN "Digikey"
+F 4 "311-1036-1-ND" H 3850 3950 50  0001 C CNN "Digikey"
 	1    3850 3950
 	1    0    0    -1
@@
 F 0 "C18" H 3625 4300 50  0000 L CNN
 F 1 "1000pF" H 3500 4225 50  0000 L CNN
-F 2 "Capacitors_SMD:C_0603" H 3850 4250 50  0001 C CNN
+F 2 "Capacitors_SMD:C_0402" H 3850 4250 50  0001 C CNN
 F 3 "" H 3850 4250 50  0001 C CNN
-F 4 "1276-1018-1-ND" H 3850 4250 50  0001 C CNN "Digikey"
+F 4 "311-1036-1-ND" H 3850 4250 50  0001 C CNN "Digikey"
 	1    3850 4250
 	1    0    0    -1
@@
 F 0 "NT3" H 5825 2700 50  0000 C CNN
 F 1 "Net-Tie_2" H 5825 2550 50  0001 C CNN
-F 2 "NetTies:NetTie-2_SMD_Pad0.5mm" H 5825 2650 50  0001 C CNN
+F 2 "MCU_Powertrain:NetTie-2_SMD_5mil" H 5825 2650 50  0001 C CNN
 F 3 "~" H 5825 2650 50  0001 C CNN
 	1    5825 2650
@@
 F 0 "NT1" H 7775 2675 50  0000 C CNN
 F 1 "Net-Tie_2" H 7775 2525 50  0001 C CNN
-F 2 "NetTies:NetTie-2_SMD_Pad0.5mm" H 7775 2625 50  0001 C CNN
+F 2 "MCU_Powertrain:NetTie-2_SMD_5mil" H 7775 2625 50  0001 C CNN
 F 3 "~" H 7775 2625 50  0001 C CNN
 	1    7775 2625
@@
 F 0 "NT2" H 9725 2675 50  0000 C CNN
 F 1 "Net-Tie_2" H 9725 2525 50  0001 C CNN
-F 2 "NetTies:NetTie-2_SMD_Pad0.5mm" H 9725 2625 50  0001 C CNN
+F 2 "MCU_Powertrain:NetTie-2_SMD_5mil" H 9725 2625 50  0001 C CNN
 F 3 "~" H 9725 2625 50  0001 C CNN
 	1    9725 2625
 	1    0    0    -1
 $EndComp
+Wire Wire Line
+	8050 2050 8050 2200
+$Comp
+L Device:Net-Tie_2 NT4
+U 1 1 5E3AFDBF
+P 7775 2200
+F 0 "NT4" H 7775 2250 50  0000 C CNN
+F 1 "Net-Tie_2" H 7775 2100 50  0001 C CNN
+F 2 "MCU_Powertrain:NetTie-2_SMD_5mil" H 7775 2200 50  0001 C CNN
+F 3 "~" H 7775 2200 50  0001 C CNN
+	1    7775 2200
+	1    0    0    -1
+$EndComp
+Wire Wire Line
+	7675 2200 7500 2200
+Wire Wire Line
+	7875 2200 8050 2200
+Connection ~ 8050 2200
+Wire Wire Line
+	8050 2200 8050 2250
+Wire Wire Line
+	9975 2050 9975 2200
+$Comp
+L Device:Net-Tie_2 NT5
+U 1 1 5E3CF519
+P 9725 2200
+F 0 "NT5" H 9725 2250 50  0000 C CNN
+F 1 "Net-Tie_2" H 9725 2100 50  0001 C CNN
+F 2 "MCU_Powertrain:NetTie-2_SMD_5mil" H 9725 2200 50  0001 C CNN
+F 3 "~" H 9725 2200 50  0001 C CNN
+	1    9725 2200
+	1    0    0    -1
+$EndComp
+Wire Wire Line
+	9625 2200 9425 2200
+Wire Wire Line
+	9825 2200 9975 2200
+Connection ~ 9975 2200
+Wire Wire Line
+	9975 2200 9975 2250
+Wire Wire Line
+	6100 2075 6100 2225
+$Comp
+L Device:Net-Tie_2 NT6
+U 1 1 5E3EF0DE
+P 5825 2225
+F 0 "NT6" H 5825 2275 50  0000 C CNN
+F 1 "Net-Tie_2" H 5825 2125 50  0001 C CNN
+F 2 "MCU_Powertrain:NetTie-2_SMD_5mil" H 5825 2225 50  0001 C CNN
+F 3 "~" H 5825 2225 50  0001 C CNN
+	1    5825 2225
+	1    0    0    -1
+$EndComp
+Wire Wire Line
+	5550 2225 5725 2225
+Wire Wire Line
+	5925 2225 6100 2225
+Connection ~ 6100 2225
+Wire Wire Line
+	6100 2225 6100 2275
 $EndSCHEMATC

Commit message: More Layout + Schematic
- Fixed small issue with net labels, ISEN labels were not seperated on the DRV sheet.
- More layout
Connections:
- net labels added: ISEN_A_DRV, ISEN_B_DRV, ISEN_C_DRV
Changed lines of the file:
@@
 $EndComp
 Wire Wire Line
-	1950 3775 1650 3775
-Wire Wire Line
-	1650 3975 1950 3975
-Wire Wire Line
-	1950 4175 1650 4175
-Text Label 1650 3775 0    50   ~ 0
-ISEN_A
-Text Label 1650 3975 0    50   ~ 0
-ISEN_B
-Text Label 1650 4175 0    50   ~ 0
-ISEN_C
+	1950 3775 1500 3775
+Wire Wire Line
+	1500 3975 1950 3975
+Wire Wire Line
+	1950 4175 1500 4175
+Text Label 1500 3775 0    50   ~ 0
+ISEN_A_DRV
+Text Label 1500 3975 0    50   ~ 0
+ISEN_B_DRV
+Text Label 1500 4175 0    50   ~ 0
+ISEN_C_DRV
 Wire Wire Line
 	1950 4475 1400 4475
@@
 	0    1    1    0
 $EndComp
-Text Label 2675 5975 2    50   ~ 0
-ISEN_A
-Wire Wire Line
-	2275 5975 2675 5975
-Wire Wire Line
-	2275 6075 2675 6075
-Wire Wire Line
-	2275 6175 2675 6175
-Text Label 2675 6075 2    50   ~ 0
-ISEN_B
-Text Label 2675 6175 2    50   ~ 0
-ISEN_C
+Text Label 2850 5975 2    50   ~ 0
+ISEN_A_DRV
+Wire Wire Line
+	2275 5975 2850 5975
+Wire Wire Line
+	2275 6075 2850 6075
+Wire Wire Line
+	2275 6175 2850 6175
+Text Label 2850 6075 2    50   ~ 0
+ISEN_B_DRV
+Text Label 2850 6175 2    50   ~ 0
+ISEN_C_DRV
 Wire Wire Line
 	3475 6025 3800 6025
@@
 P 1400 4200
 F 0 "#PWR0141" H 1400 4050 50  0001 C CNN
-F 1 "+BATT" H 1415 4373 50  0000 C CNN
+F 1 "+BATT" H 1225 4275 50  0000 C CNN
 F 2 "" H 1400 4200 50  0001 C CNN
 F 3 "" H 1400 4200 50  0001 C CNN
