File: PCBs/RPM Sensor/RPM Sensor.sch (KiCad schematic (older format))
At the start: 1 part

Commit message: Schematic + Footprints + BOM
- Completed schematic
- Assigned footprints
- Updated BOM
Parts:
- added C1, C2: 100uF, Capacitors_Tantalum_SMD:CP_Tantalum_Case-U_EIA-6032-15_Reflow, symbol Device:CP
- added C3: 0.1uF, Capacitors_SMD:C_0805, symbol Device:C_Small
- added C4: 10uF, Capacitors_SMD:C_0805, symbol Device:C_Small
- added H1, H2: MountingHole, Mounting_Holes:MountingHole_3.2mm_M3_ISO14580, symbol Mechanical:MountingHole
- added J1, J12, J3: I, Testpoints:TestPoint_Pad_D4.0mm, symbol Connector_Generic:Conn_01x01
- added J10: DO/DO, Testpoints:TestPoint_Pad_D4.0mm, symbol Connector_Generic:Conn_01x01
- added J11: SEL/SEL, Testpoints:TestPoint_Pad_D4.0mm, symbol Connector_Generic:Conn_01x01
- added J2: B, Testpoints:TestPoint_Pad_D4.0mm, symbol Connector_Generic:Conn_01x01
- added J4: A, Testpoints:TestPoint_Pad_D4.0mm, symbol Connector_Generic:Conn_01x01
- added J5: U, Testpoints:TestPoint_Pad_D4.0mm, symbol Connector_Generic:Conn_01x01
- added J6: V, Testpoints:TestPoint_Pad_D4.0mm, symbol Connector_Generic:Conn_01x01
- added J7: W/PWM, Testpoints:TestPoint_Pad_D4.0mm, symbol Connector_Generic:Conn_01x01
- added J8: SCL/CLK, Testpoints:TestPoint_Pad_D4.0mm, symbol Connector_Generic:Conn_01x01
- added J9: NSL/DI, Testpoints:TestPoint_Pad_D4.0mm, symbol Connector_Generic:Conn_01x01
- added TP1, TP10, TP11, TP12, TP13, TP14, TP15, TP16, TP2, TP3, TP4, TP5, TP6, TP7, TP8, TP9: TestPoint, Testpoints:TestPoint_Keystone_5015_Micro-Minature, symbol Connector:TestPoint
- U1: renamed from U?; footprint (none) -> Housings_DFN_QFN:QFN-24-1EP_4x4mm_Pitch0.5mm; Digikey (none) -> 516-3787-ND
Connections:
- net +5V: now also C1.1, C2.1, C3.1, C4.1, J3.1 (Pin_1), TP4.1
- net GND: now also C1.2, C2.2, C3.2, C4.2, J12.1 (Pin_1), TP13.1, TP14.1, TP15.1, TP16.1, TP5.1
- net at U1.10 (SSI_SCL_SPI_CLK): now also J8.1 (Pin_1), TP9.1
- net at U1.11 (SSI_NSL_SPI_DI): now also J9.1 (Pin_1), TP10.1
- net at U1.12 (SSI_DO_SPI_DO): now also J10.1 (Pin_1), TP11.1
- net at U1.21 (SSI_SPI_SEL): now also J11.1 (Pin_1), TP12.1
- net at U1.22 (U): now also J5.1 (Pin_1), TP6.1
- net at U1.23 (V): now also J6.1 (Pin_1), TP7.1
- net at U1.24 (W/PWM): now also J7.1 (Pin_1), TP8.1
- net at U1.7 (I): now also J1.1 (Pin_1), TP1.1
- net at U1.8 (B): now also J2.1 (Pin_1), TP2.1
- net at U1.9 (A): now also J4.1 (Pin_1), TP3.1
Other:
- note added: "place next to pins 14/13"
- note added: "place next to pins 19/20"

Commit message: Layout
- Mechanical + layout complete
Parts:
- removed TP1, TP10, TP11, TP12, TP13, TP14, TP15, TP16, TP2, TP3, TP4, TP5, TP6, TP7, TP8, TP9: TestPoint, Testpoints:TestPoint_Keystone_5015_Micro-Minature, symbol Connector:TestPoint
- added J13, J14, J15, J16: I, Testpoints:TestPoint_Pad_D2.0mm, symbol Connector_Generic:Conn_01x01
- J1, J10, J11, J12, J2, J3, J4, J5, J6, J7, J8, J9: footprint Testpoints:TestPoint_Pad_D4.0mm -> Testpoints:TestPoint_Pad_D2.0mm
Connections:
- net GND: now also J13.1 (Pin_1), J14.1 (Pin_1), J15.1 (Pin_1), J16.1 (Pin_1)

Commit message: Fixed Footprint and Gerbers
- Changed mag encoder from 4x4 to 5x5, the correct footprint. :(
- Updated Gerbers
Parts:
- U1: footprint Housings_DFN_QFN:QFN-24-1EP_4x4mm_Pitch0.5mm -> Housings_DFN_QFN:QFN-24-1EP_5x5mm_Pitch0.65mm
Changed lines of the file:
@@
 F 0 "U1" H 5550 3450 50  0000 C CNN
 F 1 "MAG_ENCODER_AEAT-8800-Q24" H 5550 1550 50  0000 C CNN
-F 2 "Housings_DFN_QFN:QFN-24-1EP_4x4mm_Pitch0.5mm" H 5400 2900 50  0001 C CNN
+F 2 "Housings_DFN_QFN:QFN-24-1EP_5x5mm_Pitch0.65mm" H 5400 2900 50  0001 C CNN
 F 3 "" H 5400 2900 50  0001 C CNN
 F 4 "516-3787-ND" H 5400 2900 50  0001 C CNN "Digikey"
