File: PCBs/Thruster_Controller/TI_MCU.sch (KiCad schematic (older format))
At the start: 14 parts, among them U5 TMS320F28027F

Commit message: Initial Routing Finished
- All layout and routing initially finished
- Still need to clean up silkscreen and any routing blemishes
Parts:
- added D5: Orange, LEDs:LED_0603, symbol Device:LED_ALT
- added R31: 680, Resistors_SMD:R_0603, symbol Device:R_US
- C34, C35, C36, C37, C38: footprint Capacitors_SMD:C_0805 -> Capacitors_SMD:C_0402; Digikey 1276-1763-1-ND -> 490-10451-1-ND
- R25, R26: footprint Resistors_SMD:R_0805 -> Resistors_SMD:R_0402; Digikey 311-820ARCT-ND -> 311-820JRCT-ND
- R27, R28, R29, R30: footprint Resistors_SMD:R_0805 -> Resistors_SMD:R_0402; Digikey 541-4139-1-ND -> 311-2.2KJRCT-ND
Connections:
- net +3V3: now also D5.2 (A)
- net GPIO33: now also R31.2
- new net: D5.1 (K), R31.1
Other:
- note added: "Test LED"
- moved on the sheet: C34, C35, C36, C37, C38, L2, L3, R25, R26, R27, R28, R29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
