File: PCBs/Thruster_Controller_V2/TI_MCU.sch (KiCad schematic (older format))
At the start: 32 parts, among them U2 TMS320F280041C, Y1 20 MHz

Commit message: Updated Footprints
- Moved over to the default KiCAD footprints, the rounded ones.
- Updated all 3D models as well
- Need to fix a bunch of DRC errors ;(
Parts:
- C16, C18, C21, C27: footprint Capacitors_SMD:C_0603 -> Capacitor_SMD:C_0603_1608Metric
- C19, C22, C29, C30, C31, C32, C33, C34, C35, C36, C37, C38, C39, C40, C41, C42: footprint Capacitors_SMD:C_0402 -> Capacitor_SMD:C_0402_1005Metric
- D5: footprint LEDs:LED_0603 -> LED_SMD:LED_0603_1608Metric
- L1, L3: footprint Inductors_SMD:L_0402 -> Inductor_SMD:L_0402_1005Metric
- R25, R26, R27, R28, R29, R30: footprint Resistors_SMD:R_0402 -> Resistor_SMD:R_0402_1005Metric
- R31: footprint Resistors_SMD:R_0603 -> Resistor_SMD:R_0603_1608Metric
- U2: footprint Housings_DFN_QFN:QFN-56-1EP_7x7mm_Pitch0.4mm -> Package_DFN_QFN:QFN-56-1EP_7x7mm_P0.4mm_EP5.6x5.6mm
Changed lines of the file:
@@
 F 0 "L3" V 1825 3000 50  0000 L CNN
 F 1 "60 Ohm" V 1700 2875 50  0000 L CNN
-F 2 "Inductors_SMD:L_0402" H 1750 3025 50  0001 C CNN
+F 2 "Inductor_SMD:L_0402_1005Metric" H 1750 3025 50  0001 C CNN
 F 3 "~" H 1750 3025 50  0001 C CNN
 F 4 "445-172882-1-ND" H 1750 3025 50  0001 C CNN "Digikey"
@@
 F 0 "U2" H 5600 4675 50  0000 C CNN
 F 1 "TMS320F280041C" H 5600 1500 50  0000 C CNN
-F 2 "Housings_DFN_QFN:QFN-56-1EP_7x7mm_Pitch0.4mm" H 5600 2825 118 0001 C CNN
+F 2 "Package_DFN_QFN:QFN-56-1EP_7x7mm_P0.4mm_EP5.6x5.6mm" H 5600 2825 118 0001 C CNN
 F 3 "http://www.ti.com/lit/ds/symlink/tms320f280041.pdf?ts=1588432897241" H 5600 2925 118 0001 C CNN
 F 4 "296-F280041CRSHSRCT-ND" H 5600 2825 50  0001 C CNN "Digikey"
@@
 F 0 "C33" H 2800 1750 50  0000 L CNN
 F 1 "0.1uF" H 2725 1600 50  0000 L CNN
-F 2 "Capacitors_SMD:C_0402" H 2975 1675 50  0001 C CNN
+F 2 "Capacitor_SMD:C_0402_1005Metric" H 2975 1675 50  0001 C CNN
 F 3 "~" H 2975 1675 50  0001 C CNN
 F 4 "490-10698-1-ND" H 2975 1675 50  0001 C CNN "Digikey"
@@
 F 0 "C31" H 2575 3650 50  0000 L CNN
 F 1 "0.1uF" H 2525 3500 50  0000 L CNN
-F 2 "Capacitors_SMD:C_0402" H 2750 3575 50  0001 C CNN
+F 2 "Capacitor_SMD:C_0402_1005Metric" H 2750 3575 50  0001 C CNN
 F 3 "~" H 2750 3575 50  0001 C CNN
 F 4 "490-10698-1-ND" H 2750 3575 50  0001 C CNN "Digikey"
@@
 F 0 "C40" H 8275 1550 50  0000 L CNN
 F 1 "0.1uF" H 8250 1400 50  0000 L CNN
-F 2 "Capacitors_SMD:C_0402" H 8250 1475 50  0001 C CNN
+F 2 "Capacitor_SMD:C_0402_1005Metric" H 8250 1475 50  0001 C CNN
 F 3 "~" H 8250 1475 50  0001 C CNN
 F 4 "490-10698-1-ND" H 8250 1475 50  0001 C CNN "Digikey"
@@
 F 0 "C34" H 2875 3750 50  0000 L CNN
 F 1 "0.1uF" H 2825 3600 50  0000 L CNN
-F 2 "Capacitors_SMD:C_0402" H 3050 3675 50  0001 C CNN
+F 2 "Capacitor_SMD:C_0402_1005Metric" H 3050 3675 50  0001 C CNN
 F 3 "~" H 3050 3675 50  0001 C CNN
 F 4 "490-10698-1-ND" H 3050 3675 50  0001 C CNN "Digikey"
@@
 F 0 "C38" H 8000 1650 50  0000 L CNN
 F 1 "0.1uF" H 7975 1500 50  0000 L CNN
-F 2 "Capacitors_SMD:C_0402" H 7975 1575 50  0001 C CNN
+F 2 "Capacitor_SMD:C_0402_1005Metric" H 7975 1575 50  0001 C CNN
 F 3 "~" H 7975 1575 50  0001 C CNN
 F 4 "490-10698-1-ND" H 7975 1575 50  0001 C CNN "Digikey"
@@
 F 0 "C41" H 8275 2850 50  0000 L CNN
 F 1 "0.1uF" H 8250 2700 50  0000 L CNN
-F 2 "Capacitors_SMD:C_0402" H 8250 2775 50  0001 C CNN
+F 2 "Capacitor_SMD:C_0402_1005Metric" H 8250 2775 50  0001 C CNN
 F 3 "~" H 8250 2775 50  0001 C CNN
 F 4 "490-10698-1-ND" H 8250 2775 50  0001 C CNN "Digikey"
@@
 F 0 "C39" H 8000 2950 50  0000 L CNN
 F 1 "0.1uF" H 7975 2800 50  0000 L CNN
-F 2 "Capacitors_SMD:C_0402" H 7975 2875 50  0001 C CNN
+F 2 "Capacitor_SMD:C_0402_1005Metric" H 7975 2875 50  0001 C CNN
 F 3 "~" H 7975 2875 50  0001 C CNN
 F 4 "490-10698-1-ND" H 7975 2875 50  0001 C CNN "Digikey"
@@
 F 0 "R30" H 3325 1325 50  0000 L CNN
 F 1 "2.2k" H 3325 1225 50  0000 L CNN
-F 2 "Resistors_SMD:R_0402" H 3275 1275 50  0001 C CNN
+F 2 "Resistor_SMD:R_0402_1005Metric" H 3275 1275 50  0001 C CNN
 F 3 "~" H 3275 1275 50  0001 C CNN
 F 4 "311-2.2KJRCT-ND" H 3275 1275 50  0001 C CNN "Digikey"
@@
 F 0 "C35" H 3100 1750 50  0000 L CNN
 F 1 "10nF" H 3050 1600 50  0000 L CNN
-F 2 "Capacitors_SMD:C_0402" H 3275 1675 50  0001 C CNN
+F 2 "Capacitor_SMD:C_0402_1005Metric" H 3275 1675 50  0001 C CNN
 F 3 "~" H 3275 1675 50  0001 C CNN
 F 4 "732-7545-1-ND" H 3275 1675 50  0001 C CNN "Digikey"
@@
 F 0 "C29" H 2350 3275 50  0000 L CNN
 F 1 "2.2uF" H 2350 3125 50  0000 L CNN
-F 2 "Capacitors_SMD:C_0402" H 2325 3200 50  0001 C CNN
+F 2 "Capacitor_SMD:C_0402_1005Metric" H 2325 3200 50  0001 C CNN
 F 3 "~" H 2325 3200 50  0001 C CNN
 F 4 "490-10451-1-ND" H 2325 3200 50  0001 C CNN "Digikey"
@@
 F 0 "C22" H 2075 3275 50  0000 L CNN
 F 1 "2.2uF" H 2075 3125 50  0000 L CNN
-F 2 "Capacitors_SMD:C_0402" H 2050 3200 50  0001 C CNN
+F 2 "Capacitor_SMD:C_0402_1005Metric" H 2050 3200 50  0001 C CNN
 F 3 "~" H 2050 3200 50  0001 C CNN
 F 4 "490-10451-1-ND" H 2050 3200 50  0001 C CNN "Digikey"
@@
 F 0 "C32" H 2925 2650 50  0000 L CNN
 F 1 "2.2uF" H 2925 2500 50  0000 L CNN
-F 2 "Capacitors_SMD:C_0402" H 2900 2575 50  0001 C CNN
+F 2 "Capacitor_SMD:C_0402_1005Metric" H 2900 2575 50  0001 C CNN
 F 3 "~" H 2900 2575 50  0001 C CNN
 F 4 "490-10451-1-ND" H 2900 2575 50  0001 C CNN "Digikey"
@@
 F 0 "C30" H 2600 2650 50  0000 L CNN
 F 1 "2.2uF" H 2600 2500 50  0000 L CNN
-F 2 "Capacitors_SMD:C_0402" H 2575 2575 50  0001 C CNN
+F 2 "Capacitor_SMD:C_0402_1005Metric" H 2575 2575 50  0001 C CNN
 F 3 "~" H 2575 2575 50  0001 C CNN
 F 4 "490-10451-1-ND" H 2575 2575 50  0001 C CNN "Digikey"
@@
 F 0 "C21" H 1500 2300 50  0000 L CNN
 F 1 "10uF" H 1475 2150 50  0000 L CNN
-F 2 "Capacitors_SMD:C_0603" H 1675 2225 50  0001 C CNN
+F 2 "Capacitor_SMD:C_0603_1608Metric" H 1675 2225 50  0001 C CNN
 F 3 "~" H 1675 2225 50  0001 C CNN
 F 4 "1276-1119-1-ND" H 1675 2225 50  0001 C CNN "Digikey"
@@
 F 0 "C27" H 2000 2300 50  0000 L CNN
 F 1 "10uF" H 1975 2150 50  0000 L CNN
-F 2 "Capacitors_SMD:C_0603" H 2175 2225 50  0001 C CNN
+F 2 "Capacitor_SMD:C_0603_1608Metric" H 2175 2225 50  0001 C CNN
 F 3 "~" H 2175 2225 50  0001 C CNN
 F 4 "1276-1119-1-ND" H 2175 2225 50  0001 C CNN "Digikey"
@@
 F 0 "L1" V 1975 1975 50  0000 L CNN
 F 1 "220 Ohm" V 1850 1825 50  0000 L CNN
-F 2 "Inductors_SMD:L_0402" H 1900 2025 50  0001 C CNN
+F 2 "Inductor_SMD:L_0402_1005Metric" H 1900 2025 50  0001 C CNN
 F 3 "~" H 1900 2025 50  0001 C CNN
 F 4 "490-11021-1-ND" H 1900 2025 50  0001 C CNN "Digikey"
@@
 F 0 "C19" H 1450 3275 50  0000 L CNN
 F 1 "2.2uF" H 1450 3125 50  0000 L CNN
-F 2 "Capacitors_SMD:C_0402" H 1425 3200 50  0001 C CNN
+F 2 "Capacitor_SMD:C_0402_1005Metric" H 1425 3200 50  0001 C CNN
 F 3 "~" H 1425 3200 50  0001 C CNN
 F 4 "490-10451-1-ND" H 1425 3200 50  0001 C CNN "Digikey"
@@
 F 0 "C18" H 2475 1750 50  0000 L CNN
 F 1 "10uF" H 2450 1600 50  0000 L CNN
-F 2 "Capacitors_SMD:C_0603" H 2650 1675 50  0001 C CNN
+F 2 "Capacitor_SMD:C_0603_1608Metric" H 2650 1675 50  0001 C CNN
 F 3 "~" H 2650 1675 50  0001 C CNN
 F 4 "1276-1119-1-ND" H 2650 1675 50  0001 C CNN "Digikey"
@@
 F 0 "C16" H 8525 2850 50  0000 L CNN
 F 1 "10uF" H 8500 2700 50  0000 L CNN
-F 2 "Capacitors_SMD:C_0603" H 8700 2775 50  0001 C CNN
+F 2 "Capacitor_SMD:C_0603_1608Metric" H 8700 2775 50  0001 C CNN
 F 3 "~" H 8700 2775 50  0001 C CNN
 F 4 "1276-1119-1-ND" H 8700 2775 50  0001 C CNN "Digikey"
@@
 F 0 "C42" H 8550 2150 50  0000 L CNN
 F 1 "0.1uF" H 8550 2000 50  0000 L CNN
-F 2 "Capacitors_SMD:C_0402" H 8525 2075 50  0001 C CNN
+F 2 "Capacitor_SMD:C_0402_1005Metric" H 8525 2075 50  0001 C CNN
 F 3 "~" H 8525 2075 50  0001 C CNN
 F 4 "490-10698-1-ND" H 8525 2075 50  0001 C CNN "Digikey"
@@
 F 0 "R25" H 1700 5150 50  0000 L CNN
 F 1 "10k" H 1675 5050 50  0000 L CNN
-F 2 "Resistors_SMD:R_0402" V 1940 5090 50  0001 C CNN
+F 2 "Resistor_SMD:R_0402_1005Metric" V 1940 5090 50  0001 C CNN
 F 3 "~" H 1900 5100 50  0001 C CNN
 F 4 "2019-RK73B1ETTP103JCT-ND" H 1900 5100 50  0001 C CNN "Digikey"
@@
 F 0 "R26" H 2000 5150 50  0000 L CNN
 F 1 "10k" H 1975 5050 50  0000 L CNN
-F 2 "Resistors_SMD:R_0402" V 2240 5090 50  0001 C CNN
+F 2 "Resistor_SMD:R_0402_1005Metric" V 2240 5090 50  0001 C CNN
 F 3 "~" H 2200 5100 50  0001 C CNN
 F 4 "2019-RK73B1ETTP103JCT-ND" H 2200 5100 50  0001 C CNN "Digikey"
@@
 F 0 "R27" H 2300 5150 50  0000 L CNN
 F 1 "2.2k" H 2275 5050 50  0000 L CNN
-F 2 "Resistors_SMD:R_0402" H 2500 5100 50  0001 C CNN
+F 2 "Resistor_SMD:R_0402_1005Metric" H 2500 5100 50  0001 C CNN
 F 3 "~" H 2500 5100 50  0001 C CNN
 F 4 "311-2.2KJRCT-ND" H 2500 5100 50  0001 C CNN "Digikey"
@@
 F 0 "R28" H 2775 5150 50  0000 L CNN
 F 1 "10k" H 2750 5050 50  0000 L CNN
-F 2 "Resistors_SMD:R_0402" V 3015 5090 50  0001 C CNN
+F 2 "Resistor_SMD:R_0402_1005Metric" V 3015 5090 50  0001 C CNN
 F 3 "~" H 2975 5100 50  0001 C CNN
 F 4 "2019-RK73B1ETTP103JCT-ND" H 2975 5100 50  0001 C CNN "Digikey"
@@
 F 0 "R29" H 3175 5150 50  0000 L CNN
 F 1 "10k" H 3150 5050 50  0000 L CNN
-F 2 "Resistors_SMD:R_0402" V 3415 5090 50  0001 C CNN
+F 2 "Resistor_SMD:R_0402_1005Metric" V 3415 5090 50  0001 C CNN
 F 3 "~" H 3375 5100 50  0001 C CNN
 F 4 "2019-RK73B1ETTP103JCT-ND" H 3375 5100 50  0001 C CNN "Digikey"
@@
 F 0 "C37" H 7050 5200 50  0000 L CNN
 F 1 "9pF" H 7050 5050 50  0000 L CNN
-F 2 "Capacitors_SMD:C_0402" H 7025 5125 50  0001 C CNN
+F 2 "Capacitor_SMD:C_0402_1005Metric" H 7025 5125 50  0001 C CNN
 F 3 "~" H 7025 5125 50  0001 C CNN
 F 4 "490-5880-1-ND" H 7025 5125 50  0001 C CNN "Digikey"
@@
 F 0 "C36" H 6450 5200 50  0000 L CNN
 F 1 "9pF" H 6450 5050 50  0000 L CNN
-F 2 "Capacitors_SMD:C_0402" H 6425 5125 50  0001 C CNN
+F 2 "Capacitor_SMD:C_0402_1005Metric" H 6425 5125 50  0001 C CNN
 F 3 "~" H 6425 5125 50  0001 C CNN
 F 4 "490-5880-1-ND" H 6425 5125 50  0001 C CNN "Digikey"
@@
 F 0 "D5" V 4689 4782 50  0000 R CNN
 F 1 "Orange" V 4598 4782 50  0000 R CNN
-F 2 "LEDs:LED_0603" H 4650 4900 50  0001 C CNN
+F 2 "LED_SMD:LED_0603_1608Metric" H 4650 4900 50  0001 C CNN
 F 3 "~" H 4650 4900 50  0001 C CNN
 F 4 "160-1180-1-ND" V 4650 4900 50  0001 C CNN "Digikey"
@@
 F 0 "R31" H 4700 5250 50  0000 L CNN
 F 1 "680" H 4700 5175 50  0000 L CNN
-F 2 "Resistors_SMD:R_0603" V 4690 5240 50  0001 C CNN
+F 2 "Resistor_SMD:R_0603_1608Metric" V 4690 5240 50  0001 C CNN
 F 3 "~" H 4650 5250 50  0001 C CNN
 F 4 "RMCF0603JT680RCT-ND" H 4650 5250 50  0001 C CNN "Digikey"
