File: PCBs/Thruster_Controller_V2/Thruster_Controller_V2.sch (KiCad schematic (older format))
At the start: 27 parts, among them J1 PHASE_A, J2 PHASE_B, J3 PHASE_C, J4 Conn_01x01, J5 Pogo Conn, J6 Conn_01x01, J7 Conn_01x01, J8 Conn_01x01, U1 NCP718AMT330, U4 NCP718BMT500, U8 ATA6561

Commit message: Updated Footprints
- Moved over to the default KiCAD footprints, the rounded ones.
- Updated all 3D models as well
- Need to fix a bunch of DRC errors ;(
Parts:
- C23: footprint Capacitors_SMD:C_0402 -> Capacitor_SMD:C_0402_1005Metric
- C28, C4, C44: footprint Capacitors_SMD:C_0603 -> Capacitor_SMD:C_0603_1608Metric
- C3, C43: footprint Capacitors_SMD:C_0805 -> Capacitor_SMD:C_0805_2012Metric
- D1, D3, D4: footprint LEDs:LED_0603 -> LED_SMD:LED_0603_1608Metric
- R19, R34: footprint Resistors_SMD:R_0603 -> Resistor_SMD:R_0603_1608Metric
- R35: footprint Resistors_SMD:R_0402 -> Resistor_SMD:R_0402_1005Metric
- R7: footprint Resistors_SMD:R_0603 -> Resistor_SMD:R_0402_1005Metric
- U1, U4: footprint Housings_DFN_QFN:DFN-6-1EP_2x2mm_Pitch0.65mm -> Package_DFN_QFN:DFN-6-1EP_2x2mm_P0.65mm_EP1x1.6mm
- U8: footprint Housings_DFN_QFN:DFN-8-1EP_3x3mm_Pitch0.65mm -> Package_DFN_QFN:DFN-8-1EP_3x3mm_P0.65mm_EP1.7x2.05mm
Changed lines of the file:
@@
 F 0 "C23" H 4575 4825 50  0000 L CNN
 F 1 "0.1uF" H 4525 4675 50  0000 L CNN
-F 2 "Capacitors_SMD:C_0402" H 4750 4750 50  0001 C CNN
+F 2 "Capacitor_SMD:C_0402_1005Metric" H 4750 4750 50  0001 C CNN
 F 3 "" H 4750 4750 50  0001 C CNN
 F 4 "490-10698-1-ND" H 4750 4750 50  0001 C CNN "Digikey"
@@
 F 0 "C28" H 4800 4825 50  0000 L CNN
 F 1 "1uF" H 4800 4675 50  0000 L CNN
-F 2 "Capacitors_SMD:C_0603" H 4950 4750 50  0001 C CNN
+F 2 "Capacitor_SMD:C_0603_1608Metric" H 4950 4750 50  0001 C CNN
 F 3 "" H 4950 4750 50  0001 C CNN
 F 4 "1276-1102-1-ND" H 4950 4750 50  0001 C CNN "Digikey"
@@
 F 0 "R35" H 6482 4979 50  0000 R CNN
 F 1 "120" H 6482 5070 50  0000 R CNN
-F 2 "Resistors_SMD:R_0402" H 6550 5025 50  0001 C CNN
+F 2 "Resistor_SMD:R_0402_1005Metric" H 6550 5025 50  0001 C CNN
 F 3 "~" H 6550 5025 50  0001 C CNN
 F 4 "311-120JRCT-ND" H 6550 5025 50  0001 C CNN "Digikey"
@@
 F 0 "U8" H 5350 4700 50  0000 C CNN
 F 1 "ATA6561" H 5925 4000 50  0000 C CNN
-F 2 "Housings_DFN_QFN:DFN-8-1EP_3x3mm_Pitch0.65mm" H 5700 3850 50  0001 C CIN
+F 2 "Package_DFN_QFN:DFN-8-1EP_3x3mm_P0.65mm_EP1.7x2.05mm" H 5700 3850 50  0001 C CIN
 F 3 "https://ww1.microchip.com/downloads/en/DeviceDoc/20005991B.pdf" H 5700 4350 50  0001 C CNN
 F 4 "ATA6561-GBQW-NCT-ND" H 5700 4350 50  0001 C CNN "Digikey"
@@
 F 0 "R7" H 3105 5490 50  0000 L CNN
 F 1 "2.7k" H 3105 5415 50  0000 L CNN
-F 2 "Resistors_SMD:R_0603" V 3095 5480 50  0001 C CNN
+F 2 "Resistor_SMD:R_0402_1005Metric" V 3095 5480 50  0001 C CNN
 F 3 "~" H 3055 5490 50  0001 C CNN
 F 4 "RMCF0603JT2K70CT-ND" H 3055 5490 50  0001 C CNN "Digikey"
@@
 F 0 "D1" V 3094 4973 50  0000 R CNN
 F 1 "BLUE" V 3003 4973 50  0000 R CNN
-F 2 "LEDs:LED_0603" H 3055 5090 50  0001 C CNN
+F 2 "LED_SMD:LED_0603_1608Metric" H 3055 5090 50  0001 C CNN
 F 3 "~" H 3055 5090 50  0001 C CNN
 F 4 "732-4966-1-ND" V 3055 5090 50  0001 C CNN "Digikey"
@@
 F 0 "D3" V 3499 4967 50  0000 R CNN
 F 1 "GREEN" V 3408 4967 50  0000 R CNN
-F 2 "LEDs:LED_0603" H 3460 5085 50  0001 C CNN
+F 2 "LED_SMD:LED_0603_1608Metric" H 3460 5085 50  0001 C CNN
 F 3 "~" H 3460 5085 50  0001 C CNN
 F 4 "732-4980-1-ND" V 3460 5085 50  0001 C CNN "Digikey"
@@
 F 0 "U1" H 1600 5500 50  0000 C CNN
 F 1 "NCP718AMT330" H 1250 4650 50  0000 C CNN
-F 2 "Housings_DFN_QFN:DFN-6-1EP_2x2mm_Pitch0.65mm" H 1575 5050 50  0001 C CNN
+F 2 "Package_DFN_QFN:DFN-6-1EP_2x2mm_P0.65mm_EP1x1.6mm" H 1575 5050 50  0001 C CNN
 F 3 "https://www.mouser.ca/datasheet/2/308/NCP718-D-1224359.pdf" H 1525 4850 50  0001 C CNN
 F 4 "NCP718AMT330TBGOSCT-ND" H 1575 5200 50  0001 C CNN "Digikey"
@@
 F 0 "C4" H 2000 5300 50  0000 L CNN
 F 1 "1uF" H 2000 5150 50  0000 L CNN
-F 2 "Capacitors_SMD:C_0603" H 2150 5225 50  0001 C CNN
+F 2 "Capacitor_SMD:C_0603_1608Metric" H 2150 5225 50  0001 C CNN
 F 3 "" H 2150 5225 50  0001 C CNN
 F 4 "1276-1102-1-ND" H 2150 5225 50  0001 C CNN "Digikey"
@@
 F 0 "C3" H 775 5300 50  0000 L CNN
 F 1 "1uF" H 725 5150 50  0000 L CNN
-F 2 "Capacitors_SMD:C_0805" H 950 5225 50  0001 C CNN
+F 2 "Capacitor_SMD:C_0805_2012Metric" H 950 5225 50  0001 C CNN
 F 3 "" H 950 5225 50  0001 C CNN
 F 4 "1276-6470-1-ND" H 950 5225 50  0001 C CNN "Digikey"
@@
 F 0 "R19" H 3510 5485 50  0000 L CNN
 F 1 "100" H 3510 5410 50  0000 L CNN
-F 2 "Resistors_SMD:R_0603" V 3500 5475 50  0001 C CNN
+F 2 "Resistor_SMD:R_0603_1608Metric" V 3500 5475 50  0001 C CNN
 F 3 "~" H 3460 5485 50  0001 C CNN
 F 4 "2019-RK73B1JTTD101JCT-ND" H 3460 5485 50  0001 C CNN "Digikey"
@@
 F 0 "U4" H 1625 7125 50  0000 C CNN
 F 1 "NCP718BMT500" H 1275 6275 50  0000 C CNN
-F 2 "Housings_DFN_QFN:DFN-6-1EP_2x2mm_Pitch0.65mm" H 1600 6675 50  0001 C CNN
+F 2 "Package_DFN_QFN:DFN-6-1EP_2x2mm_P0.65mm_EP1x1.6mm" H 1600 6675 50  0001 C CNN
 F 3 "https://www.onsemi.com/pub/Collateral/NCP718-D.PDF" H 1550 6475 50  0001 C CNN
 F 4 "NCP718BMT500TBGOSCT-ND" H 1600 6825 50  0001 C CNN "Digikey"
@@
 F 0 "C44" H 2025 6925 50  0000 L CNN
 F 1 "1uF" H 2025 6775 50  0000 L CNN
-F 2 "Capacitors_SMD:C_0603" H 2175 6850 50  0001 C CNN
+F 2 "Capacitor_SMD:C_0603_1608Metric" H 2175 6850 50  0001 C CNN
 F 3 "" H 2175 6850 50  0001 C CNN
 F 4 "1276-1102-1-ND" H 2175 6850 50  0001 C CNN "Digikey"
@@
 F 0 "C43" H 800 6925 50  0000 L CNN
 F 1 "1uF" H 750 6775 50  0000 L CNN
-F 2 "Capacitors_SMD:C_0805" H 975 6850 50  0001 C CNN
+F 2 "Capacitor_SMD:C_0805_2012Metric" H 975 6850 50  0001 C CNN
 F 3 "" H 975 6850 50  0001 C CNN
 F 4 "1276-6470-1-ND" H 975 6850 50  0001 C CNN "Digikey"
@@
 F 0 "D4" V 3939 4982 50  0000 R CNN
 F 1 "GREEN" V 3848 4982 50  0000 R CNN
-F 2 "LEDs:LED_0603" H 3900 5100 50  0001 C CNN
+F 2 "LED_SMD:LED_0603_1608Metric" H 3900 5100 50  0001 C CNN
 F 3 "~" H 3900 5100 50  0001 C CNN
 F 4 "732-4980-1-ND" V 3900 5100 50  0001 C CNN "Digikey"
@@
 F 0 "R34" H 3950 5475 50  0000 L CNN
 F 1 "220" H 3950 5400 50  0000 L CNN
-F 2 "Resistors_SMD:R_0603" V 3940 5465 50  0001 C CNN
+F 2 "Resistor_SMD:R_0603_1608Metric" V 3940 5465 50  0001 C CNN
 F 3 "~" H 3900 5475 50  0001 C CNN
 F 4 "2019-RK73B1JTTD221JCT-ND" H 3900 5475 50  0001 C CNN "Digikey"
