File: PCBs/Thruster_Controller_V2/Thruster_Controller_V2.sch (KiCad schematic (older format))
At the start: 27 parts, among them J1 PHASE_A, J2 PHASE_B, J3 PHASE_C, J4 Conn_01x01, J5 Pogo Conn, J6 Conn_01x01, J7 Conn_01x01, J8 Conn_01x01, U1 NCP718AMT330, U4 NCP718BMT500, U8 ATA6561

Commit message: New BOM
- Exported new BOM
- Updated 5V LDO PN, same thing but slight variation. Matches 3V3 PN now
Parts:
- U4: value NCP718BMT500 -> NCP718AMT500; Digikey NCP718BMT500TBGOSCT-ND -> ‎NCP718AMT500TBGOSCT-ND‎
Changed lines of the file:
@@
 P 1600 6825
 F 0 "U4" H 1625 7125 50  0000 C CNN
-F 1 "NCP718BMT500" H 1275 6275 50  0000 C CNN
+F 1 "NCP718AMT500" H 1275 6275 50  0000 C CNN
 F 2 "Package_DFN_QFN:DFN-6-1EP_2x2mm_P0.65mm_EP1x1.6mm" H 1600 6675 50  0001 C CNN
 F 3 "https://www.onsemi.com/pub/Collateral/NCP718-D.PDF" H 1550 6475 50  0001 C CNN
-F 4 "NCP718BMT500TBGOSCT-ND" H 1600 6825 50  0001 C CNN "Digikey"
+F 4 "‎NCP718AMT500TBGOSCT-ND‎" H 1600 6825 50  0001 C CNN "Digikey"
 F 5 "863-NCP718BMT500TBG" H 1600 6825 50  0001 C CNN "Mouser"
 	1    1600 6825

Commit message: Fixed a woopsies
- Change R7 from 0402 to 0603 for future board spins
Parts:
- R7: footprint Resistor_SMD:R_0402_1005Metric -> Resistor_SMD:R_0603_1608Metric
Changed lines of the file:
@@
 F 0 "R7" H 3105 5490 50  0000 L CNN
 F 1 "2.7k" H 3105 5415 50  0000 L CNN
-F 2 "Resistor_SMD:R_0402_1005Metric" V 3095 5480 50  0001 C CNN
+F 2 "Resistor_SMD:R_0603_1608Metric" V 3095 5480 50  0001 C CNN
 F 3 "~" H 3055 5490 50  0001 C CNN
 F 4 "RMCF0603JT2K70CT-ND" H 3055 5490 50  0001 C CNN "Digikey"
