File: PCBs/Thruster_Controller_V2/Thruster_Controller_V2.kicad_pcb (KiCad board)
At the start: 4 copper layers, 35.5 x 37 mm, 112 parts, among them J1 PHASE_A, J2 PHASE_B, J3 PHASE_C, J4 Conn_01x01, J5 Pogo Conn, J6 Conn_01x01, J7 Conn_01x01, J8 Conn_01x01, Q1 SIZF906DT, Q2 SIZF906DT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

Commit message: Updated Fab Layers
- Made fab layers readable for ease of use during assembly. This really comes in handy!
Parts:
- J4: value Conn_01x01 -> CANL
- J6: value Conn_01x01 -> CANH
- J7: value Conn_01x01 -> VIN
- J8: value Conn_01x01 -> GND
