File: hardware/Thruster_Controller_V2/Powertrain.sch (KiCad schematic (older format))
At the start: 53 parts, among them Q1 SIZF906DT, Q2 SIZF906DT, Q3 SIZF906DT, U3 DRV8320S

Commit message: Added Alternate Input Cap
- Added currently used 150uF, 20V input cap PN. This is probably a better selection for better input range, and 220uF might be overkill anyways.
Other:
- note added: "Or 150uF, 20V caps. PN: APXJ200ARA151MF61G"
Changed lines of the file:
@@
 Wire Wire Line
 	875  2750 875  2800
+Text Notes 6775 4100 0    50   ~ 0
+Or 150uF, 20V caps. PN: APXJ200ARA151MF61G
 $EndSCHEMATC
